File: Hardware/witnessv0.1/MCU.kicad_sch (KiCad schematic)
At the start: 8 parts, among them J1 Conn_01x02, U1 RP2354B

Commit message: esp32 mcu
Parts:
- removed U1: RP2354B, Package_DFN_QFN:QFN-80-1EP_10x10mm_P0.4mm_EP3.4x3.4mm, symbol MCU_RaspberryPi:RP2354B
- added D1: LED_RGBA, symbol Device:LED_RGBA
- added J4: Micro_SD_Card, Connector_Card:microSD_HC_Wuerth_693072010801, symbol Connector:Micro_SD_Card
- added U1: ESP32-S3FN8, Package_DFN_QFN:QFN-56-1EP_7x7mm_P0.4mm_EP4x4mm, symbol MCU_Espressif:ESP32-S3
- added U6: W25Q128JVS, Package_SO:SOIC-8_5.3x5.3mm_P1.27mm, symbol Memory_Flash:W25Q128JVS
- added Y1: F322540MUBCE2O, Crystal:Crystal_SMD_3225-4Pin_3.2x2.5mm, symbol Oscillator:ASCO
- C6: value 100n -> 1u
Connections:
- net +3V3: now reaches C5.1
- net +3V3: now also C3.1, C4.1, U1.46 (VDD3P3_CPU), U1.55 (VDDA), U1.56 (VDDA)
- net GND: now reaches C5.2
- net GND: now also C3.2, C4.2
- new net: U1.2 (VDD3P3), U1.3 (VDD3P3)
Other:
- moved on the sheet: C3, C4, C5

Commit message: power updates and some esp32 stuff
Parts:
- removed J4: Micro_SD_Card, Connector_Card:microSD_HC_Wuerth_693072010801, symbol Connector:Micro_SD_Card
- removed U6: W25Q128JVS, Package_SO:SOIC-8_5.3x5.3mm_P1.27mm, symbol Memory_Flash:W25Q128JVS
- added BZ1: Buzzer, Buzzer_Beeper:Buzzer_Murata_PKMCS0909E, symbol Device:Buzzer
- added C26, C27, C28, C29: 100n, Capacitor_SMD:C_0603_1608Metric, symbol Device:C_Small
- added C30: 1u, Capacitor_SMD:C_0603_1608Metric, symbol Device:C_Small
- added C31: 10u, Capacitor_SMD:C_0603_1608Metric, symbol Device:C_Small
- added L4: L_Small, Inductor_SMD:L_0805_2012Metric, symbol Device:L_Small
- D1: footprint (none) -> Witness:0603x2 RGB
- Y1: footprint Crystal:Crystal_SMD_3225-4Pin_3.2x2.5mm -> Oscillator:Oscillator_SMD_Abracon_ASCO-4Pin_1.6x1.2mm
Connections:
- net +3V3: now also C6.1, U1.20 (VDD3P3_RTC), U1.29 (VDD_SPI), Y1.1 (Tri-State), Y1.4 (VDD), C26.1, C27.1, C29.1, C30.1, C31.1, L4.1
- net GND: now also C6.2, Y1.2 (GND), C26.2, C27.2, C28.2, C29.2, C30.2, C31.2
- net at U1.2 (VDD3P3), U1.3 (VDD3P3): now also C28.1, L4.2
- net XIN: now reaches U1.54 (XTAL_P)
- net XIN: now also Y1.3 (OUT)
- no-connect marks 0 -> 3
Other:
- moved on the sheet: C6, Y1

Commit message: mcu updates
Parts:
- added U8: W25N01KVZEIR, Package_SON:WSON-8-1EP_8x6mm_P1.27mm_EP3.4x4.3mm, symbol Witness:W25N01KVZEIR
Connections:
- net GND: now also U1.57 (GND)
Changed lines of the file:
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@@
+	(wire
+		(pts
+			(xy 158.75 139.7) (xy 158.75 140.97)
+		)
+		(stroke
+			(width 0)
+			(type default)
+		)
+	)
 	(wire
 		(pts
@@
 	)
 	(symbol
+		(lib_id "power:GND")
+		(at 158.75 140.97 0)
+		(unit 1)
+		(body_style 1)
+		(exclude_from_sim no)
+		(in_bom yes)
+		(on_board yes)
+		(in_pos_files yes)
+		(dnp no)
+		(property "Reference" "#PWR034"
+			(at 158.75 147.32 0)
+			(hide yes)
+			(show_name no)
+			(do_not_autoplace no)
+			(effects
+				(font
+					(size 1.27 1.27)
+				)
+			)
+		)
+		(property "Value" "GND"
+			(at 158.75 145.034 0)
+			(show_name no)
+			(do_not_autoplace no)
+			(effects
+				(font
+					(size 1.27 1.27)
+				)
+			)
+		)
+		(property "Footprint" ""
+			(at 158.75 140.97 0)
+			(hide yes)
+			(show_name no)
+			(do_not_autoplace no)
+			(effects
+				(font
+					(size 1.27 1.27)
+				)
+			)
+		)
+		(property "Datasheet" ""
+			(at 158.75 140.97 0)
+			(hide yes)
+			(show_name no)
+			(do_not_autoplace no)
+			(effects
+				(font
+					(size 1.27 1.27)
+				)
+			)
+		)
+		(property "Description" "Power symbol creates a global label with name \"GND\" , ground"
+			(at 158.75 140.97 0)
+			(hide yes)
+			(show_name no)
+			(do_not_autoplace no)
+			(effects
+				(font
+					(size 1.27 1.27)
+				)
+			)
+		)
+		(pin "1"
+		)
+		(instances
+			(project "witnessv0.1"
+				(path "/c7e4a338-55e7-4896-822a-22161197db9b/84c7cad5-6a87-4e90-b655-2e6037ab0db0"
+					(reference "#PWR034")
+					(unit 1)
+				)
+			)
+		)
+	)
+	(symbol
 		(lib_id "power:+3V3")
 		(at 176.53 22.86 0)
@@
 					(unit 1)
 				)
+			)
+		)
+	)
+	(symbol
+		(lib_id "Witness:W25N01KVZEIR")
+		(at 242.57 83.82 0)
+		(unit 1)
+		(body_style 1)
+		(exclude_from_sim no)
+		(in_bom yes)
+		(on_board yes)
+		(in_pos_files yes)
+		(dnp no)
+		(fields_autoplaced yes)
+		(property "Reference" "U8"
+			(at 254 83.8199 0)
+			(show_name no)
+			(do_not_autoplace no)
+			(effects
+				(font
+					(size 1.27 1.27)
+				)
+				(justify left)
+			)
+		)
+		(property "Value" "W25N01KVZEIR"
+			(at 254 86.3599 0)
+			(show_name no)
+			(do_not_autoplace no)
+			(effects
+				(font
+					(size 1.27 1.27)
+				)
+				(justify left)
+			)
+		)
+		(property "Footprint" "Package_SON:WSON-8-1EP_8x6mm_P1.27mm_EP3.4x4.3mm"
+			(at 242.57 83.82 0)
+			(hide yes)
+			(show_name no)
+			(do_not_autoplace no)
+			(effects
+				(font
+					(size 1.27 1.27)
+				)
+			)
+		)
+		(property "Datasheet" "kicad-embed://w25n01gw revf 082418.pdf"
+			(at 242.57 83.82 0)
+			(hide yes)
+			(show_name no)
+			(do_not_autoplace no)
+			(effects
+				(font
+					(size 1.27 1.27)
+				)
+			)
+		)
+		(property "Description" ""
+			(at 242.57 83.82 0)
+			(hide yes)
+			(show_name no)
+			(do_not_autoplace no)
+			(effects
+				(font
+					(size 1.27 1.27)
+				)
+			)
+		)
+		(pin "5"
+		)
+		(pin "8"
+		)
+		(pin "7"
+		)
+		(pin "6"
+		)
+		(pin "1"
+		)
+		(pin "3"
+		)
+		(pin "4"
+		)
+		(pin "2"
+		)
+		(instances
+			(project "witnessv0.1"
+				(path "/c7e4a338-55e7-4896-822a-22161197db9b/84c7cad5-6a87-4e90-b655-2e6037ab0db0"
+					(reference "U8")
+					(unit 1)
+				)

Commit message: mcu work
Parts:
- removed C1: 100n, Capacitor_SMD:C_0603_1608Metric, symbol Device:C_Small
- added AE1: Antenna_Shield, symbol Device:Antenna_Shield
- added C32, C33: 100n, Capacitor_SMD:C_0603_1608Metric, symbol Device:C_Small
- added J4: Conn_01x02, Jumper:SolderJumper-2_P1.3mm_Open_RoundedPad1.0x1.5mm, symbol Connector_Generic:Conn_01x02
- added L5: L_Small, Inductor_SMD:L_0603_1608Metric, symbol Device:L_Small
- added R17, R18, R19, R22: 1k, Resistor_SMD:R_0603_1608Metric, symbol Device:R_Small
- added R23, R24, R25, R26, R27, R28, R29: 4.7k, Resistor_SMD:R_0603_1608Metric, symbol Device:R_Small
Connections:
- net +3V3: now also C2.1, D1.4 (A), U8.8 (VCC), R22.2, R23.2, R25.2, R26.2, R28.2
- net GND: now also BZ1.2 (-), C2.2, J1.2 (Pin_2), U8.4 (GND), AE1.2 (Shield), C32.2, C33.2, J4.2 (Pin_2), R24.1, R27.1, R29.1
- net at U1.1 (LNA_IN): now also C32.1, L5.1
- net USB_D+: now reaches U1.25 (GPIO19/USB_D-)
- net USB_D-: now reaches U1.26 (GPIO20/USB_D+)
- net SPI_HD: now reaches U1.30 (SPIHD)
- net SPI_HD: now also U8.7 (~{HOLD}/~{RESET}/IO_{3})
- net SPI_WP: now reaches U1.31 (SPIWP)
- net SPI_WP: now also U8.3 (~{WP}/IO_{2})
- net SPI_CS: now reaches U1.32 (SPICS0)
- net SPI_CS: now also U8.1 (~{CS})
- net SPI_CLK: now reaches U1.33 (SPICLK)
- net SPI_CLK: now also U8.6 (CLK)
- net SPI_Q: now reaches U1.34 (SPIQ)
- net SPI_Q: now also U8.2 (DO/IO_{1})
- net SPI_D: now reaches U1.35 (SPID)
- net SPI_D: now also U8.5 (DI/IO_{0})
- net RST: now reaches U1.4 (CHIP_PU)
- net RST: now also J1.1 (Pin_1), R22.1
- net GPIO0: now reaches U1.5 (GPIO0)
- net GPIO0: now also J4.1 (Pin_1), R23.1
- net GPIO45: now reaches U1.51 (GPIO45)
- net GPIO45: now also R26.1, R27.2
- net GPIO46: now reaches U1.52 (GPIO46)
- net GPIO46: now also R24.2, R25.1
- net GPIO3: now reaches U1.8 (GPIO3)
- net GPIO3: now also R28.1, R29.2
- net at D1.1 (RK): now also R18.2
- net at D1.2 (GK): now also R17.2
- net at D1.3 (BK): now also R19.2
- net BUZZER: now reaches BZ1.1 (+)
- new net: AE1.1 (A), C33.1, L5.2
- new net LED_B: R19.1
- new net LED_G: R17.1
- new net LED_R: R18.1
- no-connect marks 3 -> 6
Other:
- moved on the sheet: BZ1, Y1

Commit message: lots of work
Parts:
- added R30, R31: 0, Resistor_SMD:R_0603_1608Metric, symbol Device:R_Small
- AE1: footprint (none) -> Connector_Coaxial:U.FL_Molex_MCRF_73412-0110_Vertical
- L4: value L_Small -> 10n
Connections:
- net GND: no longer C29.2
- net USB_D+: now also R30.1, R31.1; no longer U1.25 (GPIO19/USB_D-)
- net USB_D-: no longer names the net of U1.26 (GPIO20/USB_D+)
- net USB_D-: now also R31.2
- new net: R30.2, U1.25 (GPIO19/USB_D-)
Other:
- note added: "INPUTS"
- note added: "OUTPUTS"
- company: (none) -> WITNESS
- title: (none) -> MCU
- moved on the sheet: C2, D1, R17, R18, R19, U8

Commit message: micro lock conenctors and sd card soldered to baord and inital palcement done.
Parts:
- removed C2: 100n, Capacitor_SMD:C_0603_1608Metric, symbol Device:C_Small
- removed U8: W25N01KVZEIR, Package_SON:WSON-8-1EP_8x6mm_P1.27mm_EP3.4x4.3mm, symbol Witness:W25N01KVZEIR
- added J10: Micro_SD_Card, microSD_Card:microSD_Card, symbol Connector:Micro_SD_Card
- C26, C27, C28, C29, C3, C30, C32, C33, C4, C5, C6: footprint Capacitor_SMD:C_0603_1608Metric -> Capacitor_SMD:C_0402_1005Metric
- L5: footprint Inductor_SMD:L_0603_1608Metric -> Inductor_SMD:L_0402_1005Metric
- R17, R18, R19, R22, R23, R24, R25, R26, R27, R28, R29, R30, R31: footprint Resistor_SMD:R_0603_1608Metric -> Resistor_SMD:R_0402_1005Metric
Connections:
- net GND: now also C29.2
- net USB_D+: no longer R30.1
- net SPI_CLK: no longer names the net of U1.33 (SPICLK)
- net SPI_CS: no longer names the net of U1.32 (SPICS0)
- net SPI_D: no longer names the net of U1.35 (SPID)
- net SPI_HD: no longer names the net of U1.30 (SPIHD)
- net SPI_Q: no longer names the net of U1.34 (SPIQ)
- net SPI_WP: no longer names the net of U1.31 (SPIWP)
- new net USB_D-: R30.1
- no-connect marks 6 -> 7
