File: Hardware/witnessv0.1/Sensors.kicad_sch (KiCad schematic)
At the start: 2 parts, among them U4 LSM6DS3, U5 ICM-20602

Commit message: esp32 mcu
Parts:
- added U7: MS5607-02BA, Package_LGA:LGA-8_3x5mm_P1.25mm, symbol Sensor_Pressure:MS5607-02BA
Connections:
- new net: U7.4 (CSB), U7.5 (CSB)
Other:
- note added: "BAROMETER"
- moved on the sheet: U4, U5
Changed lines of the file:
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@@
 	(paper "A4")
 	(rectangle
-		(start 149.86 49.53)
-		(end 256.54 151.13)
+		(start 17.78 110.49)
+		(end 109.22 189.23)
 		(stroke
 			(width 0)
@@
 	)
 	(rectangle
-		(start 33.02 50.8)
-		(end 127 152.4)
+		(start 132.08 24.13)
+		(end 226.06 101.6)
 		(stroke
 			(width 0)
@@
 		)
 	)
+	(rectangle
+		(start 16.51 24.13)
+		(end 110.49 101.6)
+		(stroke
+			(width 0)
+			(type default)
+		)
+		(fill
+			(type none)
+		)
+	)
 	(text "320G IMU"
 		(exclude_from_sim no)
-		(at 78.74 49.276 0)
+		(at 62.23 22.606 0)
 		(effects
 			(font
@@
 	(text "32G IMU"
 		(exclude_from_sim no)
-		(at 200.406 47.244 0)
+		(at 53.086 108.204 0)
 		(effects
 			(font
@@
 		)
 	)
+	(text "BAROMETER"
+		(exclude_from_sim no)
+		(at 177.8 22.606 0)
+		(effects
+			(font
+				(size 2.54 2.54)
+			)
+		)
+	)
 	(symbol
 		(lib_id "Sensor_Motion:LSM6DS3")
-		(at 81.28 90.17 0)
+		(at 50.8 54.61 0)
 		(unit 1)
 		(body_style 1)
@@
 		(fields_autoplaced yes)
 		(property "Reference" "U4"
-			(at 83.4233 105.41 0)
+			(at 52.9433 69.85 0)
 			(show_name no)
 			(do_not_autoplace no)
@@
 		)
 		(property "Value" "LSM6DS3"
-			(at 83.4233 107.95 0)
+			(at 52.9433 72.39 0)
 			(show_name no)
 			(do_not_autoplace no)
@@
 		)
 		(property "Footprint" "Package_LGA:LGA-14_3x2.5mm_P0.5mm_LayoutBorder3x4y"
-			(at 71.12 107.95 0)
+			(at 40.64 72.39 0)
 			(hide yes)
 			(show_name no)
@@
 		)
 		(property "Datasheet" "https://www.st.com/resource/en/datasheet/lsm6ds3tr-c.pdf"
-			(at 83.82 106.68 0)
+			(at 53.34 71.12 0)
 			(hide yes)
 			(show_name no)
@@
 		)
 		(property "Description" "I2C/SPI, iNEMO inertial module: always-on 3D accelerometer and 3D gyroscope"
-			(at 81.28 90.17 0)
+			(at 50.8 54.61 0)
 			(hide yes)
 			(show_name no)
@@
 	(symbol
 		(lib_id "Sensor_Motion:ICM-20602")
-		(at 203.2 91.44 0)
+		(at 62.23 137.16 0)
 		(unit 1)
 		(body_style 1)
@@
 		(fields_autoplaced yes)
 		(property "Reference" "U5"
-			(at 205.3433 104.14 0)
+			(at 64.3733 149.86 0)
 			(show_name no)
 			(do_not_autoplace no)
@@
 		)
 		(property "Value" "ICM-20602"
-			(at 205.3433 106.68 0)
+			(at 64.3733 152.4 0)
 			(show_name no)
 			(do_not_autoplace no)
@@
 		)
 		(property "Footprint" "Package_LGA:LGA-16_3x3mm_P0.5mm_LayoutBorder3x5y"
-			(at 203.2 85.09 0)
+			(at 62.23 130.81 0)
 			(hide yes)
 			(show_name no)
@@
 		)
 		(property "Datasheet" "http://www.invensense.com/wp-content/uploads/2016/10/DS-000176-ICM-20602-v1.0.pdf"
-			(at 204.47 67.31 0)
+			(at 63.5 113.03 0)
 			(hide yes)
 			(show_name no)
@@
 		)
 		(property "Description" "High performance 6-Axis MEMS motion tracking, SPI/I2C interface, LGA-16"
-			(at 203.2 91.44 0)
+			(at 62.23 137.16 0)
 			(hide yes)
 			(show_name no)
@@
 					(unit 1)
 				)
+			)
+		)
+	)
+	(symbol
+		(lib_id "Sensor_Pressure:MS5607-02BA")
+		(at 175.26 55.88 0)
+		(unit 1)
+		(body_style 1)
+		(exclude_from_sim no)
+		(in_bom yes)
+		(on_board yes)
+		(in_pos_files yes)
+		(dnp no)
+		(fields_autoplaced yes)
+		(property "Reference" "U7"
+			(at 184.15 54.6099 0)
+			(show_name no)
+			(do_not_autoplace no)
+			(effects
+				(font
+					(size 1.27 1.27)
+				)
+				(justify left)
+			)
+		)
+		(property "Value" "MS5607-02BA"
+			(at 184.15 57.1499 0)
+			(show_name no)
+			(do_not_autoplace no)
+			(effects
+				(font
+					(size 1.27 1.27)
+				)
+				(justify left)
+			)
+		)
+		(property "Footprint" "Package_LGA:LGA-8_3x5mm_P1.25mm"
+			(at 175.26 55.88 0)
+			(hide yes)
+			(show_name no)
+			(do_not_autoplace no)
+			(effects
+				(font
+					(size 1.27 1.27)
+				)
+			)
+		)
+		(property "Datasheet" "https://www.te.com/commerce/DocumentDelivery/DDEController?Action=showdoc&DocId=Data+Sheet%7FMS5607-02BA03%7FB2%7Fpdf%7FEnglish%7FENG_DS_MS5607-02BA03_B2.pdf%7FCAT-BLPS0035"
+			(at 175.26 55.88 0)
+			(hide yes)
+			(show_name no)
+			(do_not_autoplace no)
+			(effects
+				(font
+					(size 1.27 1.27)
+				)
+			)
+		)
+		(property "Description" "Barometric pressure sensor, 20cm resolution, 10 to 1200 mbar, I2C and SPI interface up to 20MHz, LGA-8"
+			(at 175.26 55.88 0)
+			(hide yes)
+			(show_name no)
+			(do_not_autoplace no)
+			(effects
+				(font
+					(size 1.27 1.27)
+				)
+			)
+		)
+		(pin "2"
+		)
+		(pin "4"
+		)
+		(pin "8"
+		)
+		(pin "1"
+		)
+		(pin "3"
+		)
+		(pin "5"
+		)
+		(pin "6"
+		)
+		(pin "7"
+		)
+		(instances
+			(project "witnessv0.1"
+				(path "/c7e4a338-55e7-4896-822a-22161197db9b/6023f714-3146-4cd2-9fdd-9f3ecdc641a0"
+					(reference "U7")
+					(unit 1)
+				)

Commit message: power updates and some esp32 stuff
Parts:
- removed U4: LSM6DS3, Package_LGA:LGA-14_3x2.5mm_P0.5mm_LayoutBorder3x4y, symbol Sensor_Motion:LSM6DS3
- removed U5: ICM-20602, Package_LGA:LGA-16_3x3mm_P0.5mm_LayoutBorder3x5y, symbol Sensor_Motion:ICM-20602
- added U4: LSM6DSV320XTR, Package_LGA:Bosch_LGA-14_3x2.5mm_P0.5mm, symbol Witness:LSM6DSV320XTR
- added U5: ICM-45686, Package_LGA:LGA-14_3x2.5mm_P0.5mm_LayoutBorder3x4y, symbol Witness:ICM-45686
Changed lines of the file:
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@@
 	)
 	(symbol
-		(lib_id "Sensor_Motion:LSM6DS3")
-		(at 50.8 54.61 0)
+		(lib_id "Witness:ICM-45686")
+		(at 64.77 148.59 0)
+		(unit 1)
+		(body_style 1)
+		(exclude_from_sim no)
+		(in_bom yes)
+		(on_board yes)
+		(in_pos_files yes)
+		(dnp no)
+		(fields_autoplaced yes)
+		(property "Reference" "U5"
+			(at 66.9133 163.83 0)
+			(show_name no)
+			(do_not_autoplace no)
+			(effects
+				(font
+					(size 1.27 1.27)
+				)
+				(justify left)
+			)
+		)
+		(property "Value" "ICM-45686"
+			(at 66.9133 166.37 0)
+			(show_name no)
+			(do_not_autoplace no)
+			(effects
+				(font
+					(size 1.27 1.27)
+				)
+				(justify left)
+			)
+		)
+		(property "Footprint" "Package_LGA:LGA-14_3x2.5mm_P0.5mm_LayoutBorder3x4y"
+			(at 64.77 148.59 0)
+			(hide yes)
+			(show_name no)
+			(do_not_autoplace no)
+			(effects
+				(font
+					(size 1.27 1.27)
+				)
+			)
+		)
+		(property "Datasheet" ""
+			(at 64.77 148.59 0)
+			(hide yes)
+			(show_name no)
+			(do_not_autoplace no)
+			(effects
+				(font
+					(size 1.27 1.27)
+				)
+			)
+		)
+		(property "Description" ""
+			(at 64.77 148.59 0)
+			(hide yes)
+			(show_name no)
+			(do_not_autoplace no)
+			(effects
+				(font
+					(size 1.27 1.27)
+				)
+			)
+		)
+		(pin "7"
+		)
+		(pin "1"
+		)
+		(pin "3"
+		)
+		(pin "5"
+		)
+		(pin "10"
+		)
+		(pin "11"
+		)
+		(pin "11"
+		)
+		(pin "7"
+		)
+		(pin "4"
+		)
+		(pin "14"
+		)
+		(pin "6"
+		)
+		(pin "9"
+		)
+		(pin "12"
+		)
+		(pin "13"
+		)
+		(pin "8"
+		)
+		(pin "2"
+		)
+		(instances
+			(project "witnessv0.1"
+				(path "/c7e4a338-55e7-4896-822a-22161197db9b/6023f714-3146-4cd2-9fdd-9f3ecdc641a0"
+					(reference "U5")
+					(unit 1)
+				)
+			)
+		)
+	)
+	(symbol
+		(lib_id "Witness:LSM6DSV320XTR")
+		(at 66.04 58.42 0)
 		(unit 1)
 		(body_style 1)
@@
 		(fields_autoplaced yes)
 		(property "Reference" "U4"
-			(at 52.9433 69.85 0)
-			(show_name no)
-			(do_not_autoplace no)
-			(effects
-				(font
-					(size 1.27 1.27)
-				)
-				(justify left)
-			)
-		)
-		(property "Value" "LSM6DS3"
-			(at 52.9433 72.39 0)
-			(show_name no)
-			(do_not_autoplace no)
-			(effects
-				(font
-					(size 1.27 1.27)
-				)
-				(justify left)
-			)
-		)
-		(property "Footprint" "Package_LGA:LGA-14_3x2.5mm_P0.5mm_LayoutBorder3x4y"
-			(at 40.64 72.39 0)
-			(hide yes)
-			(show_name no)
-			(do_not_autoplace no)
-			(effects
-				(font
-					(size 1.27 1.27)
-				)
-				(justify left)
-			)
-		)
-		(property "Datasheet" "https://www.st.com/resource/en/datasheet/lsm6ds3tr-c.pdf"
-			(at 53.34 71.12 0)
-			(hide yes)
-			(show_name no)
-			(do_not_autoplace no)
-			(effects
-				(font
-					(size 1.27 1.27)
-				)
-			)
-		)
-		(property "Description" "I2C/SPI, iNEMO inertial module: always-on 3D accelerometer and 3D gyroscope"
-			(at 50.8 54.61 0)
-			(hide yes)
-			(show_name no)
-			(do_not_autoplace no)
-			(effects
-				(font
-					(size 1.27 1.27)
-				)
-			)
+			(at 70.7233 40.64 0)
+			(show_name no)
+			(do_not_autoplace no)
+			(effects
+				(font
+					(size 1.27 1.27)
+				)
+				(justify left)
+			)
+		)
+		(property "Value" "LSM6DSV320XTR"
+			(at 70.7233 43.18 0)
+			(show_name no)
+			(do_not_autoplace no)
+			(effects
+				(font
+					(size 1.27 1.27)
+				)
+				(justify left)
+			)
+		)
+		(property "Footprint" "Package_LGA:Bosch_LGA-14_3x2.5mm_P0.5mm"
+			(at 66.04 58.42 0)
+			(hide yes)
+			(show_name no)
+			(do_not_autoplace no)
+			(effects
+				(font
+					(size 1.27 1.27)
+				)
+			)
+		)
+		(property "Datasheet" ""
+			(at 66.04 58.42 0)
+			(hide yes)
+			(show_name no)
+			(do_not_autoplace no)
+			(effects
+				(font
+					(size 1.27 1.27)
+				)
+			)
+		)
+		(property "Description" ""
+			(at 66.04 58.42 0)
+			(hide yes)
+			(show_name no)
+			(do_not_autoplace no)
+			(effects
+				(font
+					(size 1.27 1.27)
+				)
+			)
+		)
+		(pin "5"
+		)
+		(pin "7"
+		)
+		(pin "4"
+		)
+		(pin "9"
+		)
+		(pin "6"
+		)
+		(pin "10"
+		)
+		(pin "1"
+		)
+		(pin "13"
+		)
+		(pin "11"
+		)
+		(pin "12"
 		)
 		(pin "3"
 		)
-		(pin "6"
-		)
-		(pin "5"
+		(pin "8"
 		)
 		(pin "14"
 		)
-		(pin "1"
-		)
 		(pin "2"
-		)
-		(pin "4"
-		)
-		(pin "7"
-		)
-		(pin "8"
-		)
-		(pin "9"
-		)
-		(pin "10"
-		)
-		(pin "11"
-		)
-		(pin "12"
-		)
-		(pin "13"
 		)
 		(instances
@@
 					(unit 1)
 				)
-			)
-		)
-	)
-	(symbol
-		(lib_id "Sensor_Motion:ICM-20602")
-		(at 62.23 137.16 0)
-		(unit 1)
-		(body_style 1)
-		(exclude_from_sim no)
-		(in_bom yes)
-		(on_board yes)
-		(in_pos_files yes)
-		(dnp no)
-		(fields_autoplaced yes)
-		(property "Reference" "U5"
-			(at 64.3733 149.86 0)
-			(show_name no)
-			(do_not_autoplace no)
-			(effects
-				(font
-					(size 1.27 1.27)
-				)
-				(justify left)
-			)
-		)
-		(property "Value" "ICM-20602"
-			(at 64.3733 152.4 0)
-			(show_name no)
-			(do_not_autoplace no)
-			(effects
-				(font
-					(size 1.27 1.27)
-				)
-				(justify left)
-			)
-		)
-		(property "Footprint" "Package_LGA:LGA-16_3x3mm_P0.5mm_LayoutBorder3x5y"
-			(at 62.23 130.81 0)
-			(hide yes)
-			(show_name no)
-			(do_not_autoplace no)
-			(effects
-				(font
-					(size 1.27 1.27)
-				)
-			)
-		)
-		(property "Datasheet" "http://www.invensense.com/wp-content/uploads/2016/10/DS-000176-ICM-20602-v1.0.pdf"
-			(at 63.5 113.03 0)
-			(hide yes)
-			(show_name no)
-			(do_not_autoplace no)
-			(effects
-				(font
-					(size 1.27 1.27)
-				)
-			)
-		)
-		(property "Description" "High performance 6-Axis MEMS motion tracking, SPI/I2C interface, LGA-16"
-			(at 62.23 137.16 0)
-			(hide yes)
-			(show_name no)
-			(do_not_autoplace no)
-			(effects
-				(font
-					(size 1.27 1.27)
-				)
-			)
-		)
-		(pin "16"
-		)
-		(pin "14"
-		)
-		(pin "1"
-		)
-		(pin "15"
-		)
-		(pin "11"
-		)
-		(pin "13"
-		)
-		(pin "9"
-		)
-		(pin "3"
-		)
-		(pin "10"
-		)
-		(pin "6"
-		)
-		(pin "12"
-		)
-		(pin "4"
-		)
-		(pin "8"
-		)
-		(pin "5"
-		)
-		(pin "2"
-		)
-		(pin "7"
-		)
-		(instances
-			(project "witnessv0.1"
-				(path "/c7e4a338-55e7-4896-822a-22161197db9b/6023f714-3146-4cd2-9fdd-9f3ecdc641a0"
-					(reference "U5")
-					(unit 1)
-				)

Commit message: lots of work
Parts:
- added C36, C37, C38, C39, C40: 100n, Capacitor_SMD:C_0603_1608Metric, symbol Device:C_Small
Connections:
- net SPI2_CIPO: now reaches U5.1 (AP_SDO)
- net SPI2_CIPO: now also U4.1 (SDO/SA0), U7.6 (SDO)
- net SPI2_SCLK: now reaches U5.11 (RESV)
- net SPI2_SCLK: now also U4.2 (SDX), U7.8 (SCLK)
- net ICM_CS: now reaches U5.12 (AP_CS)
- net SPI2_COPI: now reaches U5.14 (AP_SDIO)
- net SPI2_COPI: now also U4.3 (SCX), U7.7 (SDI/SDA)
- net I2C_SDA: now reaches U5.2 (MAS_DA)
- net I2C_SDA: now also U4.14 (SDA)
- net I2C_SCL: now reaches U5.3 (MAS_CLK)
- net I2C_SCL: now also U4.13 (SCL)
- net ICM_INT1: now reaches U5.4 (INT1)
- net +3V3: now reaches U5.5 (VDDIO)
- net +3V3: now also U4.5 (VDDIO), U4.8 (VDD), U5.8 (VDD), U7.1 (VDD), C36.1, C37.1, C38.1, C39.1, C40.1
- net GND: now reaches U5.6 (GND)
- net GND: now also U4.6 (GND), U4.7 (GND), U7.2 (PS), U7.3 (GND), C36.2, C37.2, C38.2, C39.2, C40.2
- net ICM_INT2: now reaches U5.9 (INT2)
- net LSM_CS: now reaches U4.12 (CS)
- net LSM_INT1: now reaches U4.4 (INT1)
- net LSM_INT2: now reaches U4.9 (INT2)
- net MS56_CS: now reaches U7.4 (CSB), U7.5 (CSB)
- no-connect marks 0 -> 5
Other:
- note added: "INPUTS"
- note added: "OUTPUTS"
- company: (none) -> WITNESS
- title: (none) -> Sensors
- moved on the sheet: U5, U7

Commit message: micro lock conenctors and sd card soldered to baord and inital palcement done.
Parts:
- C36, C37, C38, C39, C40: footprint Capacitor_SMD:C_0603_1608Metric -> Capacitor_SMD:C_0402_1005Metric
Changed lines of the file:
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@@
 			)
 		)
-		(property "Footprint" "Capacitor_SMD:C_0603_1608Metric"
+		(property "Footprint" "Capacitor_SMD:C_0402_1005Metric"
 			(at 60.96 35.56 0)
 			(hide yes)
@@
 			)
 		)
-		(property "Footprint" "Capacitor_SMD:C_0603_1608Metric"
+		(property "Footprint" "Capacitor_SMD:C_0402_1005Metric"
 			(at 50.8 35.56 0)
 			(hide yes)
@@
 			)
 		)
-		(property "Footprint" "Capacitor_SMD:C_0603_1608Metric"
+		(property "Footprint" "Capacitor_SMD:C_0402_1005Metric"
 			(at 115.57 138.43 0)
 			(hide yes)
@@
 			)
 		)
-		(property "Footprint" "Capacitor_SMD:C_0603_1608Metric"
+		(property "Footprint" "Capacitor_SMD:C_0402_1005Metric"
 			(at 180.34 31.75 0)
 			(hide yes)
@@
 			)
 		)
-		(property "Footprint" "Capacitor_SMD:C_0603_1608Metric"
+		(property "Footprint" "Capacitor_SMD:C_0402_1005Metric"
 			(at 105.41 138.43 0)
 			(hide yes)
