File: Hardware/witnessv0.1/radio.kicad_sch (KiCad schematic)
At the start: 1 part, among them U3 Ai-Thinker-Ra-01

Commit message: lots of work
Parts:
- removed U3: Ai-Thinker-Ra-01, RF_Module:Ai-Thinker-Ra-01-LoRa, symbol RF_Module:Ai-Thinker-Ra-01
- added C41, C42: 100n, Capacitor_SMD:C_0603_1608Metric, symbol Device:C_Small
- added U10: RA-01SH-P, RF_Module:Ai-Thinker-Ra-01-LoRa, symbol Witness:RA-01SH-P
Connections:
- new net +3V3: C41.1, C42.1, U10.3 (VDD), U10.5 (VCC_PA)
- new net GND: C41.2, C42.2, U10.16 (GND), U10.2 (GND), U10.9 (GND)
- new net RAD_BUSY: U10.10 (BUSY)
- new net RAD_CS: U10.15 (~{NSS})
- new net RAD_DIO1: U10.6 (DIO1)
- new net RAD_RF_EN: U10.11 (RF_EN)
- new net RAD_RST: U10.4 (~{RESET})
- new net SPI1_CIPO: U10.13 (MISO)
- new net SPI1_COPI: U10.14 (MOSI)
- new net SPI1_SCLK: U10.12 (SCK)
- no-connect marks 0 -> 3
Other:
- note added: "INPUTS"
- note added: "OUTPUTS"
- note added: "Using on module ipex connector"
- company: (none) -> WITNESS
- title: (none) -> RADIO

Commit message: micro lock conenctors and sd card soldered to baord and inital palcement done.
Parts:
- added C43: 10u, Capacitor_SMD:C_0603_1608Metric, symbol Device:C_Small
- added JP6: SolderJumper_3_Open, Jumper:SolderJumper-3_P1.3mm_Open_RoundedPad1.0x1.5mm, symbol Jumper:SolderJumper_3_Open
- C41: value 100n -> 10u
- C42: footprint Capacitor_SMD:C_0603_1608Metric -> Capacitor_SMD:C_0402_1005Metric
Connections:
- net +3V3: now also JP6.1 (A); no longer U10.5 (VCC_PA)
- net GND: now also C43.1
- new net: C43.2, JP6.2 (C), U10.5 (VCC_PA)
- new net +5V: JP6.3 (B)
