File: Hardware/witnessv0.2/witness power/witnesspowerv0.2/witnesspowerv0.2.kicad_pcb (KiCad board)
At the start: 4 copper layers, 30 x 50 mm, 111 parts, among them J1 Conn_01x02, J10 Micro_SD_Card, J2 Conn_01x02, J3 USB_B_Micro, J4 Conn_01x02, J5 Conn_01x04, J6 Conn_01x04, J7 Conn_01x04, J8 Conn_01x04, J9 Conn_01x04, Q1 SQA403EJ, Q2 SQA403EJ, U1 ESP32-S3FN8, U10 RA-01SH-P, U2 TPS63070, U3 INA2180A3IDSG, U4 LSM6DSV320XTR, U5 ICM-45686, U6 TPS63070, U7 MS5607-02BA, U9 USBLC6-2SC6, Y1 F322540MUBCE2O

Commit message: trying to split it, in progress
Parts:
- removed J10: Micro_SD_Card, microSD_Card:microSD_Card
- added C35: 100n, Capacitor_SMD:C_0402_1005Metric, B.Cu at (145.7, 117.0)
- added U8: W25N01KVZEIR, Package_SON:WSON-8-1EP_8x6mm_P1.27mm_EP3.4x4.3mm, B.Cu at (140.2, 122.9)
- moved R28 11.8 mm to (131.0, 116.0)
- moved R29 11.8 mm to (131.0, 117.0)
