File: Hardware/witnessv0.2/iris/Sensors.kicad_sch (KiCad schematic)
At the start: 8 parts, among them U4 LSM6DSV320XTR, U5 ICM-45686, U7 MS5607-02BA

Commit message: iris rework
Parts:
- removed C39, C40: 100n, Capacitor_SMD:C_0402_1005Metric, symbol Device:C_Small
- removed U5: ICM-45686, Package_LGA:LGA-14_3x2.5mm_P0.5mm_LayoutBorder3x4y, symbol Witness:ICM-45686
Connections:
- net SPI2_CIPO renamed SPI3_CIPO
- net SPI2_COPI renamed SPI3_COPI
- net SPI2_SCLK renamed SPI3_SCLK
- no-connect marks 5 -> 2
Other:
- note removed: "32G IMU"
