File: Hardware/witnessv0.2/iris/radio.kicad_sch (KiCad schematic)
At the start: 5 parts, among them U10 RA-01SH-P

Commit message: iris rework
Parts:
- removed C43: 10u, Capacitor_SMD:C_0603_1608Metric, symbol Device:C_Small
- removed JP6: SolderJumper_3_Open, Jumper:SolderJumper-3_P1.3mm_Open_RoundedPad1.0x1.5mm, symbol Jumper:SolderJumper_3_Open
Connections:
- net +3V3: now also U10.5 (VCC_PA)
- net SPI1_CIPO renamed SPI3_CIPO
- net SPI1_COPI renamed SPI3_COPI
- net SPI1_SCLK renamed SPI3_SCLK
