File: Hardware/witnessv0.2/iris/IO.kicad_sch (KiCad schematic)
At the start: 17 parts, among them J2 Conn_01x02, J3 USB_B_Micro, J5 Conn_01x04, J6 Conn_01x04, J7 Conn_01x04, J8 Conn_01x04, J9 Conn_01x04, U9 USBLC6-2SC6

Commit message: iris rework
Parts:
- removed J7, J8, J9: Conn_01x04, Witness:Molex_MicroLock-2200980471-01x04-Horizontal, symbol Connector_Generic:Conn_01x04
- removed JP1, JP2, JP3, JP4, JP5: SolderJumper_3_Open, Jumper:SolderJumper-3_P1.3mm_Open_RoundedPad1.0x1.5mm, symbol Jumper:SolderJumper_3_Open
- added C28: 100n, Capacitor_SMD:C_0402_1005Metric, symbol Device:C_Small
- added R39: 120, Resistor_SMD:R_0402_1005Metric, symbol Device:R_Small
- added U5: TCAN1044A-Q1, Package_SON:VSON-8-1EP_3x3mm_P0.65mm_EP1.65x2.4mm, symbol Witness:TCAN1044A-Q1
Connections:
- net +3V3: now also J5.1 (Pin_1), C28.1, U5.3 (VCC)
- net GND: now also C28.2, U5.2 (GND)
- net USB_D+: no longer U9.3 (I/O2)
- net USB_UNSAFE_D-: now reaches J3.2 (D-), U9.4 (I/O2)
- net USB_UNSAFE_D+: now reaches J3.3 (D+), U9.6 (I/O1)
- net GPIO: now reaches J6.1 (Pin_1)
- net +BATT renamed BATT_RAW
- net GPIO1 renamed CAN_L
- net CAN_L: now also R39.1, U5.6 (CANL)
- net GPIO2 renamed CAN_H
- net CAN_H: now also R39.2, U5.7 (CANH)
- new net CANRX: U5.1 (TXD)
- new net CANTX: U5.4 (RXD)
- new net USB_D-: U9.3 (I/O2)
- no-connect marks 2 -> 4
Other:
- moved on the sheet: J5

Commit message: lots of iris work
Parts:
- added J7, J8, J9: Conn_01x04, Witness:Molex_MicroLock-2200980471-01x04-Horizontal, symbol Connector_Generic:Conn_01x04
Connections:
- net +3V3: no longer J5.1 (Pin_1)
- net GND: now also J7.4 (Pin_4), J8.4 (Pin_4), J9.4 (Pin_4)
- net RXD_MCU renamed RXD1_MCU
- net TXD_MCU renamed TXD1_MCU
- new net GPIO_P31: J8.2 (Pin_2)
- new net GPIO_P32: J8.3 (Pin_3)
- new net GPIO_P41: J9.2 (Pin_2)
- new net GPIO_P42: J9.3 (Pin_3)
- new net OUT1PWR: J5.1 (Pin_1)
- new net OUT2PWR: J7.1 (Pin_1)
- new net OUT3PWR: J8.1 (Pin_1)
- new net OUT4PWR: J9.1 (Pin_1)
- new net RXD2_MCU: J7.3 (Pin_3)
- new net TXD2_MCU: J7.2 (Pin_2)
- no-connect marks 4 -> 5
Other:
- moved on the sheet: J5, J6

Commit message: push for andrew
Parts:
- removed J9: Conn_01x04, Witness:Molex_MicroLock-2200980471-01x04-Horizontal, symbol Connector_Generic:Conn_01x04
- added R13: 0, Resistor_SMD:R_0603_1608Metric, symbol Device:R_Small
- added U3: LTV-817S, Package_DIP:SMDIP-4_W9.53mm, symbol Isolator:LTV-817S
Connections:
- net +3V3: now also R13.2
- net GPIO: no longer names the net of J6.1 (Pin_1)
- net GPIO: now also R13.1
- net GPIO_P31: no longer names the net of J8.2 (Pin_2)
- net GPIO_P31: now also U3.4
- net GPIO_P32: no longer names the net of J8.3 (Pin_3)
- net GPIO_P32: now also U3.3
- no-connect marks 5 -> 4
Other:
- moved on the sheet: C28, J8, R39, U5

Commit message: i2c io expander and repinning things
Connections:
- net RXD2_MCU is gone; now on net RXD0_MCU: J7.3 (Pin_3)
- net TXD2_MCU is gone; now on net TXD0_MCU: J7.2 (Pin_2)
Changed lines of the file:
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@@
 	(wire
 		(pts
-			(xy 41.91 54.61) (xy 44.45 54.61)
+			(xy 41.91 54.61) (xy 57.15 54.61)
 		)
 		(stroke
@@
 	(wire
 		(pts
-			(xy 41.91 52.07) (xy 44.45 52.07)
+			(xy 41.91 52.07) (xy 57.15 52.07)
 		)
 		(stroke
@@
 		)
 	)
-	(label "TXD2_MCU"
-		(at 44.45 52.07 0)
-		(effects
-			(font
-				(size 1.27 1.27)
-			)
-			(justify left bottom)
-		)
-	)
-	(label "RXD2_MCU"
-		(at 44.45 54.61 0)
-		(effects
-			(font
-				(size 1.27 1.27)
-			)
-			(justify left bottom)
-		)
-	)
 	(label "BATT_RAW"
 		(at 243.84 96.52 0)
@@
 		)
 	)
+	(label "TXD0_MCU"
+		(at 57.15 52.07 180)
+		(effects
+			(font
+				(size 1.27 1.27)
+			)
+			(justify right bottom)
+		)
+	)
 	(label "TXD1_MCU"
 		(at 245.11 36.83 0)
@@
 		)
 	)
+	(label "RXD0_MCU"
+		(at 57.15 54.61 180)
+		(effects
+			(font
+				(size 1.27 1.27)
+			)
+			(justify right bottom)
+		)
+	)

Commit message: iris inital layout
Parts:
- added R46: 1k, Resistor_SMD:R_0402_1005Metric, symbol Device:R_Small
Connections:
- net BUTTON: now also U3.1
- net GND: now also R46.2
- net at U3.2: now also R46.1
Changed lines of the file:
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@@
 	(wire
 		(pts
-			(xy 57.5931 114.3) (xy 59.69 114.3)
+			(xy 57.15 114.3) (xy 59.69 114.3)
 		)
 		(stroke
@@
 	(wire
 		(pts
-			(xy 41.91 114.3) (xy 52.5131 114.3)
+			(xy 41.91 114.3) (xy 52.07 114.3)
 		)
 		(stroke
@@
 	(wire
 		(pts
+			(xy 90.17 86.36) (xy 90.17 88.9)
+		)
+		(stroke
+			(width 0)
+			(type default)
+		)
+	)
+	(wire
+		(pts
 			(xy 135.89 181.61) (xy 135.89 177.8)
 		)
@@
 	(wire
 		(pts
+			(xy 85.09 76.2) (xy 99.06 76.2)
+		)
+		(stroke
+			(width 0)
+			(type default)
+		)
+	)
+	(wire
+		(pts
 			(xy 41.91 35.56) (xy 44.45 35.56)
 		)
@@
 		(pts
 			(xy 59.69 121.92) (xy 41.91 121.92)
+		)
+		(stroke
+			(width 0)
+			(type default)
+		)
+	)
+	(wire
+		(pts
+			(xy 85.09 81.28) (xy 90.17 81.28)
 		)
 		(stroke
@@
 			)
 			(justify left bottom)
+		)
+	)
+	(label "BUTTON"
+		(at 99.06 76.2 180)
+		(effects
+			(font
+				(size 1.27 1.27)
+			)
+			(justify right bottom)
 		)
 	)
@@
 				(path "/c7e4a338-55e7-4896-822a-22161197db9b/5a3b15b3-53d3-4c9c-a1c0-f7e9d04d876d"
 					(reference "#PWR057")
+					(unit 1)
+				)
+			)
+		)
+	)
+	(symbol
+		(lib_id "Device:R_Small")
+		(at 90.17 83.82 0)
+		(unit 1)
+		(body_style 1)
+		(exclude_from_sim no)
+		(in_bom yes)
+		(on_board yes)
+		(in_pos_files yes)
+		(dnp no)
+		(property "Reference" "R46"
+			(at 87.376 83.82 0)
+			(show_name no)
+			(do_not_autoplace no)
+			(effects
+				(font
+					(size 1.016 1.016)
+				)
+			)
+		)
+		(property "Value" "1k"
+			(at 92.202 83.82 0)
+			(show_name no)
+			(do_not_autoplace no)
+			(effects
+				(font
+					(size 1.27 1.27)
+				)
+			)
+		)
+		(property "Footprint" "Resistor_SMD:R_0402_1005Metric"
+			(at 90.17 83.82 0)
+			(hide yes)
+			(show_name no)
+			(do_not_autoplace no)
+			(effects
+				(font
+					(size 1.27 1.27)
+				)
+			)
+		)
+		(property "Datasheet" ""
+			(at 90.17 83.82 0)
+			(hide yes)
+			(show_name no)
+			(do_not_autoplace no)
+			(effects
+				(font
+					(size 1.27 1.27)
+				)
+			)
+		)
+		(property "Description" "Resistor, small symbol"
+			(at 90.17 83.82 0)
+			(hide yes)
+			(show_name no)
+			(do_not_autoplace no)
+			(effects
+				(font
+					(size 1.27 1.27)
+				)
+			)
+		)
+		(property "LCSC_Part" "C11702"
+			(at 90.17 83.82 0)
+			(hide yes)
+			(show_name no)
+			(do_not_autoplace no)
+			(effects
+				(font
+					(size 1.27 1.27)
+				)
+			)
+		)
+		(pin "2"
+		)
+		(pin "1"
+		)
+		(instances
+			(project "iris"
+				(path "/c7e4a338-55e7-4896-822a-22161197db9b/5a3b15b3-53d3-4c9c-a1c0-f7e9d04d876d"
+					(reference "R46")
 					(unit 1)
 				)
@@
 	(symbol
 		(lib_id "Device:R_Small")
-		(at 55.0531 114.3 90)
+		(at 54.61 114.3 90)
 		(unit 1)
 		(body_style 1)
@@
 		(fields_autoplaced yes)
 		(property "Reference" "R13"
-			(at 55.0531 109.22 90)
+			(at 54.61 109.22 90)
 			(show_name no)
 			(do_not_autoplace no)
@@
 		)
 		(property "Value" "0"
-			(at 55.0531 111.76 90)
+			(at 54.61 111.76 90)
 			(show_name no)
 			(do_not_autoplace no)
@@
 		)
 		(property "Footprint" "Resistor_SMD:R_0603_1608Metric"
-			(at 55.0531 114.3 0)
+			(at 54.61 114.3 0)
 			(hide yes)
 			(show_name no)
@@
 		)
 		(property "Datasheet" ""
-			(at 55.0531 114.3 0)
+			(at 54.61 114.3 0)
 			(hide yes)
 			(show_name no)
@@
 		)
 		(property "Description" "Resistor, small symbol"
-			(at 55.0531 114.3 0)
+			(at 54.61 114.3 0)
 			(hide yes)
 			(show_name no)
@@
 					(unit 1)
 				)
+			)
+		)
+	)
+	(symbol
+		(lib_id "power:GND")
+		(at 90.17 88.9 0)
+		(mirror y)
+		(unit 1)
+		(body_style 1)
+		(exclude_from_sim no)
+		(in_bom yes)
+		(on_board yes)
+		(in_pos_files yes)
+		(dnp no)
+		(fields_autoplaced yes)
+		(property "Reference" "#PWR066"
+			(at 90.17 95.25 0)
+			(hide yes)
+			(show_name no)
+			(do_not_autoplace no)
+			(effects
+				(font
+					(size 1.27 1.27)
+				)
+			)
+		)
+		(property "Value" "GND"
+			(at 90.17 93.98 0)
+			(show_name no)
+			(do_not_autoplace no)
+			(effects
+				(font
+					(size 1.27 1.27)
+				)
+			)
+		)
+		(property "Footprint" ""
+			(at 90.17 88.9 0)
+			(hide yes)
+			(show_name no)
+			(do_not_autoplace no)
+			(effects
+				(font
+					(size 1.27 1.27)
+				)
+			)
+		)
+		(property "Datasheet" ""
+			(at 90.17 88.9 0)
+			(hide yes)
+			(show_name no)
+			(do_not_autoplace no)
+			(effects
+				(font
+					(size 1.27 1.27)
+				)
+			)
+		)
+		(property "Description" "Power symbol creates a global label with name \"GND\" , ground"
+			(at 90.17 88.9 0)
+			(hide yes)
+			(show_name no)
+			(do_not_autoplace no)
+			(effects
+				(font
+					(size 1.27 1.27)
+				)
+			)
+		)
+		(pin "1"
+		)
+		(instances
+			(project "iris"
+				(path "/c7e4a338-55e7-4896-822a-22161197db9b/5a3b15b3-53d3-4c9c-a1c0-f7e9d04d876d"
+					(reference "#PWR066")
+					(unit 1)
+				)

Commit message: routed
Parts:
- added R47: 0, Resistor_SMD:R_0402_1005Metric, symbol Device:R_Small
Connections:
- net BUTTON: now also U3.2; no longer U3.1
- net GND: now also R47.1
- net at R46.1: now also U3.1; no longer U3.2
- net at J8.2 (Pin_2): now also U3.3; no longer U3.4
- net at J8.3 (Pin_3): now also U3.4; no longer U3.3
- net at J3.SH (Shield): now also R47.2
- no-connect marks 4 -> 3
Other:
- moved on the sheet: U3
Changed lines of the file:
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@@
 	)
 	(junction
+		(at 213.36 138.43)
+		(diameter 0)
+		(color 0 0 0 0)
+	)
+	(junction
 		(at 163.83 68.58)
 		(diameter 0)
@@
 	)
 	(no_connect
-		(at 210.82 132.08)
-	)
-	(no_connect
 		(at 176.53 102.87)
 	)
@@
 	(wire
 		(pts
+			(xy 213.36 138.43) (xy 213.36 139.7)
+		)
+		(stroke
+			(width 0)
+			(type default)
+		)
+	)
+	(wire
+		(pts
 			(xy 245.11 77.47) (xy 257.81 77.47)
 		)
@@
 	(wire
 		(pts
+			(xy 210.82 138.43) (xy 213.36 138.43)
+		)
+		(stroke
+			(width 0)
+			(type default)
+		)
+	)
+	(wire
+		(pts
 			(xy 250.19 121.92) (xy 262.89 121.92)
 		)
@@
 	(wire
 		(pts
-			(xy 213.36 132.08) (xy 213.36 135.89)
+			(xy 213.36 132.08) (xy 213.36 138.43)
 		)
 		(stroke
@@
 	(wire
 		(pts
+			(xy 210.82 132.08) (xy 210.82 133.35)
+		)
+		(stroke
+			(width 0)
+			(type default)
+		)
+	)
+	(wire
+		(pts
 			(xy 85.09 81.28) (xy 90.17 81.28)
 		)
@@
 	)
 	(symbol
+		(lib_id "Device:R_Small")
+		(at 210.82 135.89 180)
+		(unit 1)
+		(body_style 1)
+		(exclude_from_sim no)
+		(in_bom yes)
+		(on_board yes)
+		(in_pos_files yes)
+		(dnp no)
+		(property "Reference" "R47"
+			(at 212.598 135.89 90)
+			(show_name no)
+			(do_not_autoplace no)
+			(effects
+				(font
+					(size 1.016 1.016)
+				)
+			)
+		)
+		(property "Value" "0"
+			(at 209.042 135.89 90)
+			(show_name no)
+			(do_not_autoplace no)
+			(effects
+				(font
+					(size 1.27 1.27)
+				)
+			)
+		)
+		(property "Footprint" "Resistor_SMD:R_0402_1005Metric"
+			(at 210.82 135.89 0)
+			(hide yes)
+			(show_name no)
+			(do_not_autoplace no)
+			(effects
+				(font
+					(size 1.27 1.27)
+				)
+			)
+		)
+		(property "Datasheet" ""
+			(at 210.82 135.89 0)
+			(hide yes)
+			(show_name no)
+			(do_not_autoplace no)
+			(effects
+				(font
+					(size 1.27 1.27)
+				)
+			)
+		)
+		(property "Description" "Resistor, small symbol"
+			(at 210.82 135.89 0)
+			(hide yes)
+			(show_name no)
+			(do_not_autoplace no)
+			(effects
+				(font
+					(size 1.27 1.27)
+				)
+			)
+		)
+		(property "LCSC_Part" "C17168"
+			(at 210.82 135.89 90)
+			(hide yes)
+			(show_name no)
+			(do_not_autoplace no)
+			(effects
+				(font
+					(size 1.27 1.27)
+				)
+			)
+		)
+		(pin "2"
+		)
+		(pin "1"
+		)
+		(instances
+			(project "iris"
+				(path "/c7e4a338-55e7-4896-822a-22161197db9b/5a3b15b3-53d3-4c9c-a1c0-f7e9d04d876d"
+					(reference "R47")
+					(unit 1)
+				)
+			)
+		)
+	)
+	(symbol
 		(lib_id "power:GND")
 		(at 245.11 130.81 0)
@@
 	(symbol
 		(lib_id "power:GND")
-		(at 213.36 135.89 0)
+		(at 213.36 139.7 0)
 		(unit 1)
 		(body_style 1)
@@
 		(fields_autoplaced yes)
 		(property "Reference" "#PWR010"
-			(at 213.36 142.24 0)
+			(at 213.36 146.05 0)
 			(hide yes)
 			(show_name no)
@@
 		)
 		(property "Value" "GND"
-			(at 213.36 140.97 0)
+			(at 213.36 144.78 0)
 			(show_name no)
 			(do_not_autoplace no)
@@
 		)
 		(property "Footprint" ""
-			(at 213.36 135.89 0)
+			(at 213.36 139.7 0)
 			(hide yes)
 			(show_name no)
@@
 		)
 		(property "Datasheet" ""
-			(at 213.36 135.89 0)
+			(at 213.36 139.7 0)
 			(hide yes)
 			(show_name no)
@@
 		)
 		(property "Description" "Power symbol creates a global label with name \"GND\" , ground"
-			(at 213.36 135.89 0)
+			(at 213.36 139.7 0)
 			(hide yes)
 			(show_name no)
@@
 	(symbol
 		(lib_id "Isolator:LTV-817S")
-		(at 77.47 78.74 0)
-		(mirror y)
+		(at 77.47 78.74 180)
 		(unit 1)
 		(body_style 1)
@@
 		(dnp no)
 		(property "Reference" "U3"
-			(at 77.47 69.85 0)
+			(at 77.47 87.63 0)
 			(show_name no)
 			(do_not_autoplace no)
@@
 		)
 		(property "Value" "LTV-817S"
-			(at 77.47 72.39 0)
+			(at 77.47 85.09 0)
 			(show_name no)
 			(do_not_autoplace no)
@@
 		)
 		(property "Footprint" "Package_DIP:SMDIP-4_W9.53mm"
-			(at 77.47 86.36 0)
+			(at 77.47 71.12 0)
 			(hide yes)
 			(show_name no)
@@
 		)
 		(property "Datasheet" "http://www.us.liteon.com/downloads/LTV-817-827-847.PDF"
-			(at 86.36 71.12 0)
+			(at 86.36 86.36 0)
 			(hide yes)
 			(show_name no)

Commit message: root feedback
Parts:
- added R51: 0, Resistor_SMD:R_0402_1005Metric, symbol Device:R_Small
- R13: LCSC_Part (none) -> C21189
Connections:
- net GND: now also R51.1
- net at U5.8 (STB): now also R51.2
- no-connect marks 3 -> 2
Other:
- moved on the sheet: C28, J6, R13, R39, U5

Commit message: updates from folks
Connections:
- net USB_UNSAFE_D+ is gone; now on net USB_D+: J3.3 (D+), U9.6 (I/O1)
- net USB_UNSAFE_D- is gone; now on net USB_D-: J3.2 (D-), U9.4 (I/O2)
- net BUTTON: now also U3.1; no longer U3.2
- net at R46.1: now also U3.2; no longer U3.1
Other:
- moved on the sheet: J3, R47, U9
