File: Hardware/witnessv0.2/iris/iris.kicad_pcb (KiCad board)
At the start: 4 copper layers, 20 x 40 mm, 104 parts, among them J1 Conn_01x02, J2 Conn_01x02, J3 USB_B_Micro, J4 Conn_01x02, J5 Conn_01x04, J6 Conn_01x04, J7 Conn_01x04, J8 Conn_01x04, Q1 SQA403EJ, Q11 AO3400A, Q12 SQA403EJ, Q2 SQA403EJ, Q3 SQA403EJ, Q4 AO3400A, Q5 AO3400A, Q6 SQA403EJ, U1 PAC1934x-xJQ, U2 ME6118A33PG, U3 LTV-817S, U4 MCP23008-xML, U5 TCAN1044A-Q1, U6 TPS63070, U7 ESP32-C3FH4, U9 USBLC6-2SC6, Y1 F322540MUBCE2O

Commit message: iris release
Parts:
- removed R42, R45: 1k, Resistor_SMD:R_0402_1005Metric
- added R25: 4.7k, Resistor_SMD:R_0402_1005Metric, B.Cu at (108.6, 111.3)
- added R26: 4.7k, Resistor_SMD:R_0402_1005Metric, B.Cu at (108.6, 110.3)
Connections:
- J4 pad 1: /MCU/LED_G -> /MCU/LS_EN
- R23 pad 1: /MCU/LED_G -> /MCU/LS_EN
Routing:
- net /MCU/LED_G: track 12.9 -> 4.99 mm, vias 1 -> 0
- net /MCU/LS_EN: track 46.1 -> 48.7 mm, vias 2 -> 3
