File: Hardware/witnessv0.2/iris/loadswitches.kicad_sch (KiCad schematic)
At the start: 19 parts, among them Q11 AO3400A, Q12 SQA403EJ, Q13 AO3400A, Q14 SQA403EJ, Q3 SQA403EJ, Q4 AO3400A, Q5 AO3400A, Q6 SQA403EJ, U1 PAC1934x-xJQ

Commit message: push for andrew
Parts:
- removed Q13: AO3400A, Package_TO_SOT_SMD:SOT-23, symbol Transistor_FET:AO3400A
- removed Q14: SQA403EJ, Package_TO_SOT_SMD:Vishay_PowerPAK_SC70-6L_Single, symbol Witness:SQA403EJ
- removed R50: 1k, Resistor_SMD:R_0402_1005Metric, symbol Device:R_Small
- removed R51: 20m, Resistor_SMD:R_0603_1608Metric, symbol Device:R_Small
Connections:
- net CS2: now also Q12.1 (D), R49.2; no longer Q3.1 (D), R43.2
- net CS3: now also Q3.1 (D), R43.2; no longer Q12.1 (D), R49.2
- net EN1: no longer Q11.1 (G)
- net EN2: now also Q11.1 (G)
- net EN3: now also Q4.1 (G)
- net GND: now also U1.1 (SLOW), U1.16 (~{PWRDN})
- net VIN1: no longer R43.1, R49.1, U1.10 (SENSE4+)
- net VIN2: now also R49.1
- net VIN3: now also R43.1
- net VOUT1: no longer Q12.4 (S), Q3.4 (S)
- net VOUT2: now also Q12.4 (S), Q3.4 (S)
- net CS4: no longer names the net of U1.9 (SENSE4-)
- no-connect marks 0 -> 2

Commit message: i2c io expander and repinning things
Parts:
- added R50, R51, R52: 10k, Resistor_SMD:R_0402_1005Metric, symbol Device:R_Small
Connections:
- net EN1: now also R51.2
- net EN2: now also R50.2
- net EN3: now also R52.2
- net GND: now also R50.1, R51.1, R52.1

Commit message: iris inital layout
Parts:
- removed R50, R51: 10k, Resistor_SMD:R_0402_1005Metric, symbol Device:R_Small
- added R53, R54: 10k, Resistor_SMD:R_0402_1005Metric, symbol Device:R_Small
- R52: LCSC_Part C11702 -> (none)
Connections:
- net EN1: now also R54.2
- net EN2: now also R53.2
- net GND: now also R53.1, R54.1
- net VOUT2: no longer Q3.4 (S)
- new net VOUT3: Q3.4 (S)
Other:
- note added: "High Side Load Switch 1"
- note added: "High Side Load Switch 2"
- note added: "High Side Load Switch 3"
- note added: "I2C Current Moniter"
- moved on the sheet: C8, Q11, Q12, Q3, Q4, R40, R43, R48, R49, R52, U1

Commit message: routed
Connections:
- net +3V3: now also U1.16 (~{PWRDN})
- net CS1: now also U1.7 (SENSE3-); no longer U1.12 (SENSE1-)
- net CS3: now also U1.12 (SENSE1-); no longer U1.7 (SENSE3-)
- net GND: no longer U1.16 (~{PWRDN})
- net VIN1: no longer U1.11 (SENSE1+), U1.13 (SENSE2+)
- net VIN2: now also U1.13 (SENSE2+)
- net VIN3: now also U1.11 (SENSE1+)

Commit message: root feedback
Parts:
- R43, R44, R49: LCSC_Part (none) -> C911681
- R52, R53, R54: LCSC_Part (none) -> C25744
- U1: LCSC_Part (none) -> C623960
Other:
- moved on the sheet: Q3, Q4, R40, R43, R52

Commit message: updates from folks
Connections:
- net VIN1: now also R41.2
- net VIN2: now also R48.2
- net VIN3: now also R40.2
- removed net +5V: R40.2, R41.2, R48.2
