File: Hardware/witnessv0.2/witness/Sensors.kicad_sch (KiCad schematic)
At the start: 5 parts, among them U4 LSM6DSV320XTR, U7 MS5607-02BA

Commit message: routed
Connections:
- net I2C_SCL is gone; now on net SPI3_SCLK: U4.13 (SCL)
- net I2C_SDA is gone; now on net SPI3_COPI: U4.14 (SDA)
- net GND: now also U4.2 (SDX), U4.3 (SCX)
- net SPI3_COPI: no longer U4.3 (SCX)
- net SPI3_SCLK: no longer U4.2 (SDX)
Changed lines of the file:
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@@
 	)
 	(junction
+		(at 48.26 54.61)
+		(diameter 0)
+		(color 0 0 0 0)
+	)
+	(junction
 		(at 66.04 31.75)
 		(diameter 0)
@@
 	(wire
 		(pts
-			(xy 50.8 60.96) (xy 41.91 60.96)
+			(xy 144.78 44.45) (xy 165.1 44.45)
 		)
 		(stroke
@@
 	(wire
 		(pts
-			(xy 144.78 44.45) (xy 165.1 44.45)
+			(xy 81.28 50.8) (xy 91.44 50.8)
 		)
 		(stroke
@@
 	(wire
 		(pts
-			(xy 81.28 50.8) (xy 91.44 50.8)
+			(xy 246.38 25.4) (xy 260.35 25.4)
 		)
 		(stroke
@@
 	(wire
 		(pts
-			(xy 246.38 25.4) (xy 260.35 25.4)
+			(xy 60.96 31.75) (xy 66.04 31.75)
 		)
 		(stroke
@@
 	(wire
 		(pts
-			(xy 60.96 31.75) (xy 66.04 31.75)
+			(xy 60.96 38.1) (xy 60.96 39.37)
 		)
 		(stroke
@@
 	(wire
 		(pts
-			(xy 60.96 38.1) (xy 60.96 39.37)
+			(xy 262.89 64.77) (xy 247.65 64.77)
 		)
 		(stroke
@@
 	(wire
 		(pts
-			(xy 262.89 64.77) (xy 247.65 64.77)
+			(xy 48.26 53.34) (xy 50.8 53.34)
+		)
+		(stroke
+			(width 0)
+			(type default)
+		)
+	)
+	(wire
+		(pts
+			(xy 50.8 55.88) (xy 48.26 55.88)
 		)
 		(stroke
@@
 	(wire
 		(pts
+			(xy 30.48 58.42) (xy 30.48 54.61)
+		)
+		(stroke
+			(width 0)
+			(type default)
+		)
+	)
+	(wire
+		(pts
 			(xy 180.34 34.29) (xy 180.34 35.56)
 		)
@@
 	(wire
 		(pts
+			(xy 48.26 54.61) (xy 48.26 55.88)
+		)
+		(stroke
+			(width 0)
+			(type default)
+		)
+	)
+	(wire
+		(pts
 			(xy 66.04 77.47) (xy 67.31 77.47)
 		)
@@
 	(wire
 		(pts
-			(xy 36.83 50.8) (xy 50.8 50.8)
+			(xy 30.48 54.61) (xy 48.26 54.61)
 		)
 		(stroke
@@
 	(wire
 		(pts
-			(xy 36.83 53.34) (xy 50.8 53.34)
+			(xy 175.26 39.37) (xy 175.26 29.21)
 		)
 		(stroke
@@
 	(wire
 		(pts
-			(xy 36.83 55.88) (xy 50.8 55.88)
+			(xy 60.96 33.02) (xy 60.96 31.75)
 		)
 		(stroke
@@
 	(wire
 		(pts
-			(xy 175.26 39.37) (xy 175.26 29.21)
+			(xy 50.8 38.1) (xy 50.8 39.37)
 		)
 		(stroke
@@
 	(wire
 		(pts
-			(xy 60.96 33.02) (xy 60.96 31.75)
+			(xy 36.83 50.8) (xy 50.8 50.8)
 		)
 		(stroke
@@
 	(wire
 		(pts
-			(xy 50.8 38.1) (xy 50.8 39.37)
+			(xy 36.83 63.5) (xy 50.8 63.5)
 		)
 		(stroke
@@
 	(wire
 		(pts
-			(xy 50.8 63.5) (xy 41.91 63.5)
+			(xy 36.83 60.96) (xy 50.8 60.96)
 		)
 		(stroke
@@
 	(wire
 		(pts
-			(xy 246.38 40.64) (xy 260.35 40.64)
-		)
-		(stroke
-			(width 0)
-			(type default)
-		)
-	)
-	(wire
-		(pts
 			(xy 67.31 73.66) (xy 67.31 77.47)
 		)
@@
 	(wire
 		(pts
-			(xy 260.35 38.1) (xy 246.38 38.1)
+			(xy 68.58 41.91) (xy 68.58 43.18)
 		)
 		(stroke
@@
 	(wire
 		(pts
-			(xy 68.58 41.91) (xy 68.58 43.18)
+			(xy 151.13 54.61) (xy 165.1 54.61)
 		)
 		(stroke
@@
 	(wire
 		(pts
-			(xy 151.13 54.61) (xy 165.1 54.61)
+			(xy 48.26 54.61) (xy 48.26 53.34)
 		)
 		(stroke
@@
 		)
 	)
-	(label "LSM_CS"
-		(at 246.38 31.75 0)
+	(label "SPI3_SCLK"
+		(at 36.83 63.5 0)
 		(effects
 			(font
@@
 		)
 	)
-	(label "I2C_SCL"
-		(at 246.38 38.1 0)
+	(label "LSM_CS"
+		(at 246.38 31.75 0)
 		(effects
 			(font
@@
 		)
 	)
-	(label "I2C_SDA"
-		(at 41.91 60.96 0)
-		(effects
-			(font
-				(size 1.27 1.27)
-			)
-			(justify left bottom)
-		)
-	)
 	(label "SPI3_COPI"
 		(at 151.13 49.53 0)
@@
 	)
 	(label "SPI3_SCLK"
-		(at 36.83 53.34 0)
-		(effects
-			(font
-				(size 1.27 1.27)
-			)
-			(justify left bottom)
-		)
-	)
-	(label "SPI3_SCLK"
 		(at 151.13 52.07 0)
 		(effects
@@
 		)
 	)
-	(label "SPI3_COPI"
-		(at 36.83 55.88 0)
-		(effects
-			(font
-				(size 1.27 1.27)
-			)
-			(justify left bottom)
-		)
-	)
-	(label "I2C_SDA"
-		(at 246.38 40.64 0)
+	(label "SPI3_CIPO"
+		(at 36.83 50.8 0)
 		(effects
 			(font
@@
 		)
 	)
-	(label "LSM_INT1"
-		(at 91.44 50.8 180)
+	(label "SPI3_COPI"
+		(at 36.83 60.96 0)
 		(effects
 			(font
 				(size 1.27 1.27)
 			)
-			(justify right bottom)
+			(justify left bottom)
 		)
 	)
-	(label "SPI3_CIPO"
-		(at 36.83 50.8 0)
+	(label "LSM_INT1"
+		(at 91.44 50.8 180)
 		(effects
 			(font
 				(size 1.27 1.27)
 			)
-			(justify left bottom)
+			(justify right bottom)
 		)
 	)
@@
 		)
 	)
-	(label "I2C_SCL"
-		(at 41.91 63.5 0)
-		(effects
-			(font
-				(size 1.27 1.27)
-			)
-			(justify left bottom)
-		)
-	)
 	(label "LSM_CS"
 		(at 41.91 66.04 0)
@@
 		)
 	)
-	(hierarchical_label "I2C_SDA"
-		(shape bidirectional)
-		(at 260.35 40.64 0)
-		(effects
-			(font
-				(size 1.27 1.27)
-			)
-			(justify left)
-		)
-	)
-	(hierarchical_label "I2C_SCL"
-		(shape input)
-		(at 260.35 38.1 0)
-		(effects
-			(font
-				(size 1.27 1.27)
-			)
-			(justify left)
-		)
-	)
 	(hierarchical_label "MS56_CS"
 		(shape input)
@@
 					(unit 1)
 				)
+			)
+		)
+	)
+	(symbol
+		(lib_id "power:GND")
+		(at 30.48 58.42 0)
+		(unit 1)
+		(body_style 1)
+		(exclude_from_sim no)
+		(in_bom yes)
+		(on_board yes)
+		(in_pos_files yes)
+		(dnp no)
+		(fields_autoplaced yes)
+		(property "Reference" "#PWR063"
+			(at 30.48 64.77 0)
+			(hide yes)
+			(show_name no)
+			(do_not_autoplace no)
+			(effects
+				(font
+					(size 1.27 1.27)
+				)
+			)
+		)
+		(property "Value" "GND"
+			(at 30.48 63.5 0)
+			(show_name no)
+			(do_not_autoplace no)
+			(effects
+				(font
+					(size 1.27 1.27)
+				)
+			)
+		)
+		(property "Footprint" ""
+			(at 30.48 58.42 0)
+			(hide yes)
+			(show_name no)
+			(do_not_autoplace no)
+			(effects
+				(font
+					(size 1.27 1.27)
+				)
+			)
+		)
+		(property "Datasheet" ""
+			(at 30.48 58.42 0)
+			(hide yes)
+			(show_name no)
+			(do_not_autoplace no)
+			(effects
+				(font
+					(size 1.27 1.27)
+				)
+			)
+		)
+		(property "Description" "Power symbol creates a global label with name \"GND\" , ground"
+			(at 30.48 58.42 0)
+			(hide yes)
+			(show_name no)
+			(do_not_autoplace no)
+			(effects
+				(font
+					(size 1.27 1.27)
+				)
+			)
+		)
+		(pin "1"
+		)
+		(instances
+			(project "witness"
+				(path "/c7e4a338-55e7-4896-822a-22161197db9b/6023f714-3146-4cd2-9fdd-9f3ecdc641a0"
+					(reference "#PWR063")
+					(unit 1)
+				)
