File: Hardware/witnessv0.2/witness/radio.kicad_sch (KiCad schematic)
At the start: 3 parts, among them U10 RA-01SH-P

Commit message: routed
Connections:
- net RAD_DIO2: now reaches U10.7 (DIO2)
- net RAD_DIO3: now reaches U10.8 (DIO3)
- no-connect marks 3 -> 1
Changed lines of the file:
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@@
 	(rectangle
 		(start 233.68 12.7)
-		(end 284.48 40.64)
+		(end 284.48 45.72)
 		(stroke
 			(width 0)
@@
 	)
 	(rectangle
-		(start 233.68 40.64)
-		(end 284.48 60.96)
+		(start 233.68 45.72)
+		(end 284.48 66.04)
 		(stroke
 			(width 0)
@@
 	(text "OUTPUTS"
 		(exclude_from_sim no)
-		(at 258.064 42.672 0)
+		(at 258.064 47.752 0)
 		(effects
 			(font
@@
 	)
 	(no_connect
-		(at 160.02 88.9)
-	)
-	(no_connect
-		(at 160.02 86.36)
-	)
-	(no_connect
 		(at 160.02 76.2)
 	)
@@
 	(wire
 		(pts
+			(xy 160.02 88.9) (xy 172.72 88.9)
+		)
+		(stroke
+			(width 0)
+			(type default)
+		)
+	)
+	(wire
+		(pts
 			(xy 160.02 83.82) (xy 172.72 83.82)
 		)
@@
 	(wire
 		(pts
-			(xy 251.46 49.53) (xy 237.49 49.53)
+			(xy 251.46 54.61) (xy 237.49 54.61)
 		)
 		(stroke
@@
 	(wire
 		(pts
-			(xy 248.92 36.83) (xy 234.95 36.83)
+			(xy 248.92 41.91) (xy 234.95 41.91)
+		)
+		(stroke
+			(width 0)
+			(type default)
+		)
+	)
+	(wire
+		(pts
+			(xy 234.95 34.29) (xy 248.92 34.29)
 		)
 		(stroke
@@
 	(wire
 		(pts
-			(xy 248.92 34.29) (xy 234.95 34.29)
-		)
-		(stroke
-			(width 0)
-			(type default)
-		)
-	)
-	(wire
-		(pts
 			(xy 129.54 93.98) (xy 139.7 93.98)
 		)
@@
 	(wire
 		(pts
+			(xy 160.02 86.36) (xy 172.72 86.36)
+		)
+		(stroke
+			(width 0)
+			(type default)
+		)
+	)
+	(wire
+		(pts
 			(xy 125.73 81.28) (xy 139.7 81.28)
 		)
@@
 		(pts
 			(xy 148.59 58.42) (xy 148.59 59.69)
+		)
+		(stroke
+			(width 0)
+			(type default)
+		)
+	)
+	(wire
+		(pts
+			(xy 234.95 36.83) (xy 248.92 36.83)
+		)
+		(stroke
+			(width 0)
+			(type default)
+		)
+	)
+	(wire
+		(pts
+			(xy 234.95 39.37) (xy 248.92 39.37)
 		)
 		(stroke
@@
 		)
 	)
+	(label "RAD_DIO2"
+		(at 234.95 36.83 0)
+		(effects
+			(font
+				(size 1.27 1.27)
+			)
+			(justify left bottom)
+		)
+	)
+	(label "RAD_DIO1"
+		(at 172.72 83.82 180)
+		(effects
+			(font
+				(size 1.27 1.27)
+			)
+			(justify right bottom)
+		)
+	)
+	(label "RAD_DIO3"
+		(at 234.95 39.37 0)
+		(effects
+			(font
+				(size 1.27 1.27)
+			)
+			(justify left bottom)
+		)
+	)
 	(label "SPI3_CIPO"
 		(at 234.95 22.86 0)
@@
 	)
 	(label "RAD_BUSY"
-		(at 237.49 49.53 0)
+		(at 237.49 54.61 0)
 		(effects
 			(font
@@
 		)
 	)
+	(label "RAD_DIO2"
+		(at 172.72 86.36 180)
+		(effects
+			(font
+				(size 1.27 1.27)
+			)
+			(justify right bottom)
+		)
+	)
 	(label "RAD_RST"
 		(at 129.54 93.98 0)
@@
 		)
 	)
+	(label "RAD_DIO1"
+		(at 234.95 34.29 0)
+		(effects
+			(font
+				(size 1.27 1.27)
+			)
+			(justify left bottom)
+		)
+	)
 	(label "RAD_RST"
 		(at 234.95 31.75 0)
@@
 		)
 	)
+	(label "RAD_DIO3"
+		(at 172.72 88.9 180)
+		(effects
+			(font
+				(size 1.27 1.27)
+			)
+			(justify right bottom)
+		)
+	)
 	(label "RAD_RF_EN"
-		(at 234.95 36.83 0)
+		(at 234.95 41.91 0)
 		(effects
 			(font
@@
 		)
 	)
-	(label "RAD_DIO1"
-		(at 172.72 83.82 180)
-		(effects
-			(font
-				(size 1.27 1.27)
-			)
-			(justify right bottom)
-		)
-	)
 	(label "RAD_BUSY"
 		(at 172.72 93.98 180)
@@
 			)
 			(justify right bottom)
-		)
-	)
-	(label "RAD_DIO1"
-		(at 234.95 34.29 0)
-		(effects
-			(font
-				(size 1.27 1.27)
-			)
-			(justify left bottom)
 		)
 	)
@@
 		)
 	)
+	(hierarchical_label "RAD_DIO2"
+		(shape input)
+		(at 248.92 36.83 0)
+		(effects
+			(font
+				(size 1.27 1.27)
+			)
+			(justify left)
+		)
+	)
 	(hierarchical_label "RAD_BUSY"
 		(shape output)
-		(at 251.46 49.53 0)
+		(at 251.46 54.61 0)
 		(effects
 			(font
@@
 		)
 	)
+	(hierarchical_label "RAD_DIO3"
+		(shape input)
+		(at 248.92 39.37 0)
+		(effects
+			(font
+				(size 1.27 1.27)
+			)
+			(justify left)
+		)
+	)
 	(hierarchical_label "SPI3_COPI"
 		(shape input)
@@
 		)
 	)
+	(hierarchical_label "RAD_RF_EN"
+		(shape input)
+		(at 248.92 41.91 0)
+		(effects
+			(font
+				(size 1.27 1.27)
+			)
+			(justify left)
+		)
+	)
 	(hierarchical_label "RAD_DIO1"
 		(shape input)
@@
 		(effects
 			(font
-				(size 1.27 1.27)
-			)
-			(justify left)
-		)
-	)
-	(hierarchical_label "RAD_RF_EN"
-		(shape input)
-		(at 248.92 36.83 0)
-		(effects
-			(font
