File: Hardware/witnessv0.2/witness/MCU.kicad_sch (KiCad schematic)
At the start: 33 parts, among them J1 Conn_01x02, J4 Conn_01x02, U1 ESP32-S3FN8, U8 W25N01KVZEIR, Y1 F322540MUBCE2O

Commit message: iris rework
Connections:
- net BUZZER: now also U1.36 (SPICLK_N)
- net LED_B: now also U1.37 (SPICLK_P)
- net LED_G: now also U1.48 (MTMS)
- net LED_R: now also U1.47 (MTDI)
- net RAD_BUSY: now also U1.44 (MTCK)
- net RAD_DIO1: now also U1.7 (GPIO2)
- net RAD_RF_EN: now also U1.45 (MTDO)
- net RAD_RST: now also U1.11 (GPIO6)
Changed lines of the file:
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@@
 	)
 	(no_connect
-		(at 181.61 88.9)
-	)
-	(no_connect
-		(at 181.61 91.44)
+		(at 181.61 119.38)
 	)
 	(no_connect
@@
 		(at 181.61 73.66)
 	)
+	(no_connect
+		(at 181.61 121.92)
+	)
 	(wire
 		(pts
@@
 	(wire
 		(pts
+			(xy 194.31 106.68) (xy 181.61 106.68)
+		)
+		(stroke
+			(width 0)
+			(type default)
+		)
+	)
+	(wire
+		(pts
 			(xy 137.16 54.61) (xy 132.08 54.61)
 		)
@@
 	(wire
 		(pts
+			(xy 181.61 116.84) (xy 191.77 116.84)
+		)
+		(stroke
+			(width 0)
+			(type default)
+		)
+	)
+	(wire
+		(pts
 			(xy 252.73 120.65) (xy 252.73 128.27)
 		)
@@
 	(wire
 		(pts
+			(xy 135.89 76.2) (xy 123.19 76.2)
+		)
+		(stroke
+			(width 0)
+			(type default)
+		)
+	)
+	(wire
+		(pts
 			(xy 31.75 64.77) (xy 26.67 64.77)
 		)
@@
 	(wire
 		(pts
-			(xy 205.74 121.92) (xy 212.09 121.92)
-		)
-		(stroke
-			(width 0)
-			(type default)
-		)
-	)
-	(wire
-		(pts
 			(xy 257.81 25.4) (xy 245.11 25.4)
 		)
@@
 	(wire
 		(pts
-			(xy 194.31 106.68) (xy 181.61 106.68)
-		)
-		(stroke
-			(width 0)
-			(type default)
-		)
-	)
-	(wire
-		(pts
 			(xy 124.46 114.3) (xy 135.89 114.3)
 		)
@@
 	(wire
 		(pts
-			(xy 222.25 86.36) (xy 208.28 86.36)
-		)
-		(stroke
-			(width 0)
-			(type default)
-		)
-	)
-	(wire
-		(pts
 			(xy 181.61 127) (xy 190.5 127)
 		)
@@
 	(wire
 		(pts
-			(xy 205.74 111.76) (xy 212.09 111.76)
+			(xy 147.32 163.83) (xy 151.13 163.83)
 		)
 		(stroke
@@
 	(wire
 		(pts
-			(xy 147.32 163.83) (xy 151.13 163.83)
+			(xy 181.61 91.44) (xy 191.77 91.44)
 		)
 		(stroke
@@
 	(wire
 		(pts
+			(xy 181.61 88.9) (xy 191.77 88.9)
+		)
+		(stroke
+			(width 0)
+			(type default)
+		)
+	)
+	(wire
+		(pts
 			(xy 187.96 43.18) (xy 198.12 43.18)
 		)
@@
 	(wire
 		(pts
+			(xy 121.92 86.36) (xy 135.89 86.36)
+		)
+		(stroke
+			(width 0)
+			(type default)
+		)
+	)
+	(wire
+		(pts
 			(xy 187.96 50.8) (xy 187.96 49.53)
 		)
@@
 	(wire
 		(pts
+			(xy 181.61 114.3) (xy 191.77 114.3)
+		)
+		(stroke
+			(width 0)
+			(type default)
+		)
+	)
+	(wire
+		(pts
+			(xy 195.58 111.76) (xy 181.61 111.76)
+		)
+		(stroke
+			(width 0)
+			(type default)
+		)
+	)
+	(wire
+		(pts
 			(xy 166.37 168.91) (xy 161.29 168.91)
 		)
@@
 	(wire
 		(pts
-			(xy 95.25 175.26) (xy 99.06 175.26)
+			(xy 195.58 109.22) (xy 181.61 109.22)
 		)
 		(stroke
@@
 	(wire
 		(pts
-			(xy 205.74 116.84) (xy 212.09 116.84)
+			(xy 95.25 175.26) (xy 99.06 175.26)
 		)
 		(stroke
@@
 	(wire
 		(pts
-			(xy 222.25 95.25) (xy 208.28 95.25)
-		)
-		(stroke
-			(width 0)
-			(type default)
-		)
-	)
-	(wire
-		(pts
 			(xy 166.37 166.37) (xy 166.37 168.91)
 		)
@@
 	(wire
 		(pts
-			(xy 208.28 90.17) (xy 222.25 90.17)
-		)
-		(stroke
-			(width 0)
-			(type default)
-		)
-	)
-	(wire
-		(pts
-			(xy 222.25 92.71) (xy 208.28 92.71)
-		)
-		(stroke
-			(width 0)
-			(type default)
-		)
-	)
-	(wire
-		(pts
 			(xy 111.76 24.13) (xy 101.6 24.13)
 		)
@@
 		)
 	)
+	(label "RAD_DIO1"
+		(at 123.19 76.2 0)
+		(effects
+			(font
+				(size 1.27 1.27)
+			)
+			(justify left bottom)
+		)
+	)
 	(label "XIN"
 		(at 125.73 129.54 0)
@@
 	)
 	(label "RAD_BUSY"
-		(at 208.28 86.36 0)
+		(at 195.58 109.22 180)
 		(effects
 			(font
 				(size 1.27 1.27)
 			)
-			(justify left bottom)
+			(justify right bottom)
 		)
 	)
@@
 		)
 	)
-	(label "LED_B"
-		(at 205.74 121.92 0)
-		(effects
-			(font
-				(size 1.27 1.27)
-			)
-			(justify left bottom)
-		)
-	)
 	(label "LED_R"
-		(at 205.74 111.76 0)
+		(at 191.77 114.3 180)
 		(effects
 			(font
 				(size 1.27 1.27)
 			)
-			(justify left bottom)
+			(justify right bottom)
 		)
 	)
@@
 	)
 	(label "RAD_RF_EN"
-		(at 208.28 95.25 0)
+		(at 195.58 111.76 180)
 		(effects
 			(font
 				(size 1.27 1.27)
 			)
-			(justify left bottom)
+			(justify right bottom)
 		)
 	)
 	(label "LED_G"
-		(at 205.74 116.84 0)
+		(at 191.77 116.84 180)
 		(effects
 			(font
 				(size 1.27 1.27)
 			)
-			(justify left bottom)
+			(justify right bottom)
 		)
 	)
@@
 		)
 	)
+	(label "RAD_RST"
+		(at 121.92 86.36 0)
+		(effects
+			(font
+				(size 1.27 1.27)
+			)
+			(justify left bottom)
+		)
+	)
+	(label "LED_B"
+		(at 191.77 91.44 180)
+		(effects
+			(font
+				(size 1.27 1.27)
+			)
+			(justify right bottom)
+		)
+	)
 	(label "SPI2_IO3"
 		(at 232.41 146.05 0)
@@
 	)
 	(label "GPIO"
-		(at 181.61 106.68 0)
+		(at 194.31 106.68 180)
 		(effects
 			(font
 				(size 1.27 1.27)
 			)
-			(justify left bottom)
+			(justify right bottom)
 		)
 	)
@@
 		)
 	)
+	(label "BUZZER"
+		(at 191.77 88.9 180)
+		(effects
+			(font
+				(size 1.27 1.27)
+			)
+			(justify right bottom)
+		)
+	)
 	(label "TXD_MCU"
 		(at 245.11 59.69 0)
@@
 		)
 	)
-	(label "RAD_DIO1"
-		(at 208.28 92.71 0)
-		(effects
-			(font
-				(size 1.27 1.27)
-			)
-			(justify left bottom)
-		)
-	)
 	(label "FLASH_CS"
 		(at 125.73 96.52 0)
@@
 		(effects
 			(font
-				(size 1.27 1.27)
-			)
-			(justify left bottom)
-		)
-	)
-	(label "RAD_RST"
-		(at 208.28 90.17 0)
-		(effects
-			(font

Commit message: for foo & root
Parts:
- added D6: BZX584C10, Diode_SMD:D_SOD-523, symbol Device:D_Zener_Small
- added Q11: AO3400A, Package_TO_SOT_SMD:SOT-23, symbol Transistor_FET:AO3400A
Connections:
- net +3V3: now also BZ1.1 (+), D6.1 (K)
- net BUZZER: now also Q11.1 (G); no longer BZ1.1 (+)
- net GND: now also Q11.2 (S); no longer BZ1.2 (-)
- new net: BZ1.2 (-), D6.2 (A), Q11.3 (D)
Other:
- moved on the sheet: BZ1

Commit message: routed
Parts:
- added C7: 100n, Capacitor_SMD:C_0402_1005Metric, symbol Device:C_Small
Connections:
- net I2C_SCL is gone; now on net LED_G: U1.39 (GPIO34)
- net I2C_SDA is gone; now on net LED_R: U1.38 (GPIO33)
- net +3V3: now also C7.1
- net GND: now also C7.2
- net LED_G: no longer U1.48 (MTMS)
- net LED_R: no longer U1.47 (MTDI)
- net LSM_INT1: now also U1.47 (MTDI); no longer U1.12 (GPIO7)
- net LSM_INT2: now also U1.48 (MTMS); no longer U1.13 (GPIO8)
- net RAD_DIO1: now also U1.12 (GPIO7); no longer U1.7 (GPIO2)
- net RAD_RST: now also U1.13 (GPIO8); no longer U1.11 (GPIO6)
- net GPIO: no longer names the net of U1.43 (GPIO38)
- new net RAD_DIO2: U1.11 (GPIO6)
- new net RAD_DIO3: U1.7 (GPIO2)
- no-connect marks 10 -> 11
Other:
- moved on the sheet: C35, U8

Commit message: root feedback
Parts:
- C32, C33: now not fitted
- L5: value L_Small -> 0
Changed lines of the file:
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@@
 		(on_board yes)
 		(in_pos_files yes)
-		(dnp no)
+		(dnp yes)
 		(fields_autoplaced yes)
 		(property "Reference" "C32"
@@
 		(on_board yes)
 		(in_pos_files yes)
-		(dnp no)
+		(dnp yes)
 		(fields_autoplaced yes)
 		(property "Reference" "C33"
@@
 			)
 		)
-		(property "Value" "L_Small"
+		(property "Value" "0"
 			(at 195.58 139.7 90)
 			(show_name no)

Commit message: updates from folks
Parts:
- Le1: renamed from L5; LCSC_Part C77103 -> (none)
Other:
- moved on the sheet: C30, C31
