File: Hardware/witnessv0.2/witness/witness.kicad_sch (KiCad schematic)
At the start: 4 parts

Commit message: routed
Other:
- sheet IO ports: added none; removed GPIO
- sheet MCU ports: added RAD_DIO2, RAD_DIO3; removed GPIO, I2C_SCL, I2C_SDA
- sheet Radio ports: added RAD_DIO2, RAD_DIO3; removed none
- sheet Sensors ports: added none; removed I2C_SCL, I2C_SDA

Commit message: schematic notes on the sheets
Other:
- note added: "ESP32-C3 MCU 3x 2A load switches that can either source 5V power from a 5v Buck Boost or raw battery. current monitoring on all channels CAN to talk to the rest of the vehicle avionics. optocoupler to "push" the button on a gopro to start and end recording."
Changed lines of the file:
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@@
 		(company "WITNESS")
+	)
+	(rectangle
+		(start 58.42 19.05)
+		(end 198.12 40.64)
+		(stroke
+			(width 0)
+			(type default)
+		)
+		(fill
+			(type none)
+		)
+	)
+	(text "ESP32-C3 MCU\n3x 2A load switches that can either source 5V power from a 5v Buck Boost or raw battery. \ncurrent monitoring on all channels  \nCAN to talk to the rest of the vehicle avionics. \noptocoupler to \"push\" the button on a gopro to start and end recording.\n"
+		(exclude_from_sim no)
+		(at 59.182 30.226 0)
+		(effects
+			(font
+				(size 1.905 1.905)
+			)
+			(justify left)
+		)
 	)
 	(junction
