File: Hardware/witnessv0.2/witness/witness.kicad_sch (KiCad schematic)
At the start: 4 parts

Commit message: witness release
Other:
- note added: "ESP32-S3 for compute, LSM6DSV320P IMU for +-320G accel, +-32G accel, and 4000dps gyro MS5607 Barometer UART output for attaching an external GPS module 800mW radio module for downlink 1gbit of flash storage for flight data CAN to talk to the rest of the vehicle"
- note removed: "ESP32-C3 MCU 3x 2A load switches that can either source 5V power from a 5v Buck Boost or raw battery. current monitoring on all channels CAN to talk to the rest of the vehicle avionics. optocoupler to "push" the button on a gopro to start and end recording."
Changed lines of the file:
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@@
 	)
 	(rectangle
-		(start 58.42 19.05)
-		(end 198.12 40.64)
+		(start 83.82 17.78)
+		(end 199.39 43.18)
 		(stroke
 			(width 0)
-			(type default)
+			(type solid)
 		)
 		(fill
@@
 		)
 	)
-	(text "ESP32-C3 MCU\n3x 2A load switches that can either source 5V power from a 5v Buck Boost or raw battery. \ncurrent monitoring on all channels  \nCAN to talk to the rest of the vehicle avionics. \noptocoupler to \"push\" the button on a gopro to start and end recording.\n"
+	(text "ESP32-S3 for compute, \nLSM6DSV320P IMU for +-320G accel, +-32G accel, and 4000dps gyro \nMS5607 Barometer\nUART output for attaching an external GPS module \n800mW radio module for downlink\n1gbit of flash storage for flight data\nCAN to talk to the rest of the vehicle"
 		(exclude_from_sim no)
-		(at 59.182 30.226 0)
+		(at 84.582 30.226 0)
 		(effects
 			(font
