File: Hardware/witnessv0.2/witness/IO.kicad_sch (KiCad schematic)
At the start: 12 parts, among them J2 Conn_01x02, J3 USB_B_Micro, J5 Conn_01x04, J6 Conn_01x04, U5 TCAN1044A-Q1, U9 USBLC6-2SC6

Commit message: iris rework
Connections:
- net USB_D+: no longer U9.3 (I/O2)
- net USB_UNSAFE_D-: now reaches J3.2 (D-), U9.4 (I/O2)
- net USB_UNSAFE_D+: now reaches J3.3 (D+), U9.6 (I/O1)
- new net USB_D-: U9.3 (I/O2)
Changed lines of the file:
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@@
+		)
+	)
+	(label "USB_UNSAFE_D+"
+		(at 237.49 121.92 180)
+		(effects
+			(font
+				(size 1.27 1.27)
+			)
+			(justify right bottom)
+		)
+	)
+	(label "USB_UNSAFE_D-"
+		(at 237.49 124.46 180)
+		(effects
+			(font
+				(size 1.27 1.27)
+			)
+			(justify right bottom)
 		)
 	)
@@
 	(hierarchical_label "USB_D+"
 		(shape bidirectional)
-		(at 257.81 29.21 0)
+		(at 257.81 31.75 0)
 		(effects
 			(font
@@
 	(hierarchical_label "USB_D-"
 		(shape bidirectional)
-		(at 257.81 31.75 0)
-		(effects
-			(font
+		(at 257.81 29.21 0)
+		(effects
+			(font

Commit message: routed
Parts:
- added R13: 0, Resistor_SMD:R_0603_1608Metric, symbol Device:R_Small
- added R38: 0, Resistor_SMD:R_0402_1005Metric, symbol Device:R_Small
Connections:
- net +3V3: now also R13.2
- net GND: now also R38.1
- net at J3.SH (Shield): now also R38.2
- net GPIO: no longer names the net of J6.1 (Pin_1)
- net GPIO: now also R13.1
- no-connect marks 4 -> 3

Commit message: root feedback
Parts:
- added R51: 0, Resistor_SMD:R_0402_1005Metric, symbol Device:R_Small
Connections:
- net GND: now also R51.1
- net at U5.8 (STB): now also R51.2
- no-connect marks 3 -> 2
Other:
- moved on the sheet: C28, J6, R13, R39, U5

Commit message: updates from folks
Connections:
- net USB_UNSAFE_D+ is gone; now on net USB_D+: J3.3 (D+), U9.6 (I/O1)
- net USB_UNSAFE_D- is gone; now on net USB_D-: J3.2 (D-), U9.4 (I/O2)
Changed lines of the file:
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@@
+	)
+	(junction
+		(at 240.03 121.92)
+		(diameter 0)
+		(color 0 0 0 0)
+	)
+	(junction
+		(at 240.03 124.46)
+		(diameter 0)
+		(color 0 0 0 0)
 	)
 	(junction
@@
 	)
 	(junction
+		(at 250.19 124.46)
+		(diameter 0)
+		(color 0 0 0 0)
+	)
+	(junction
 		(at 68.58 93.98)
+		(diameter 0)
+		(color 0 0 0 0)
+	)
+	(junction
+		(at 250.19 121.92)
 		(diameter 0)
 		(color 0 0 0 0)
@@
 	(wire
 		(pts
+			(xy 240.03 121.92) (xy 250.19 121.92)
+		)
+		(stroke
+			(width 0)
+			(type default)
+		)
+	)
+	(wire
+		(pts
 			(xy 135.89 162.56) (xy 139.7 162.56)
 		)
@@
 		)
 		(stroke
+			(width 0)
+			(type default)
+		)
+	)
+	(wire
+		(pts
+			(xy 240.03 124.46) (xy 250.19 124.46)
+		)
+		(stroke

Commit message: witness release
Parts:
- R51: LCSC_Part C11702 -> C17168
Changed lines of the file:
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@@
-		)
-	)
-	(label "USB_UNSAFE_D+"
-		(at 237.49 121.92 180)
-		(effects
-			(font
-				(size 1.27 1.27)
-			)
-			(justify right bottom)
-		)
-	)
-	(label "USB_UNSAFE_D-"
-		(at 237.49 124.46 180)
-		(effects
-			(font
-				(size 1.27 1.27)
-			)
-			(justify right bottom)
 		)
 	)
@@
 			)
 		)
-		(property "LCSC_Part" "C11702"
+		(property "LCSC_Part" "C17168"
 			(at 120.65 105.41 0)
 			(hide yes)
