File: Hardware/witnessv0.2/witness/witness.kicad_pcb (KiCad board)
At the start: 4 copper layers, 20 x 40 mm, 67 parts, among them J1 Conn_01x02, J2 Conn_01x02, J3 USB_B_Micro, J4 Conn_01x02, J5 Conn_01x04, J6 Conn_01x04, Q1 SQA403EJ, Q2 SQA403EJ, U1 ESP32-S3FN8, U10 RA-01SH-P, U2 ME6118A33PG, U4 LSM6DSV320XTR, U5 TCAN1044A-Q1, U7 MS5607-02BA, U8 W25N01KVZEIR, U9 USBLC6-2SC6, Y1 F322540MUBCE2O

Commit message: iris rework
Parts:
- moved R39 7.83 mm to (119.1, 132.9), turned to 90 degrees
- moved C26 6.69 mm to (115.6, 111.1)
- moved R33 6.51 mm to (115.4, 124.4), turned to 180 degrees
- moved R34 5.88 mm to (115.4, 125.7), turned to 0 degrees
- moved C28 5.12 mm to (120.2, 126.8)
- moved R31 4.90 mm to (114.5, 116.1)
- moved R30 4.90 mm to (115.6, 116.1)
- moved U9 1.49 mm to (115.6, 119.3), turned to -90 degrees
- moved C32 1.35 mm to (107.8, 106.5)
- moved C33 1.35 mm to (107.8, 103.7)
- moved J3 1.10 mm to (121.5, 121.0)
- moved C27 0.90 mm to (113.5, 116.8)
- moved C6 0.90 mm to (112.5, 116.8)
- moved R20 0.49 mm to (106.8, 127.3)
- moved C4 0.40 mm to (105.4, 108.2)
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Connections:
- net Net-(J3-D+) renamed /IO/USB_UNSAFE_D+
- net Net-(J3-D-) renamed /IO/USB_UNSAFE_D-
- R30 pad 1: /IO/USB_D+ -> /IO/USB_D-
- U1 pad 11: unconnected-(U1-GPIO6-Pad11) -> /MCU/RAD_RST
- U1 pad 36: unconnected-(U1-SPICLK_N-Pad36) -> /MCU/BUZZER
- U1 pad 37: unconnected-(U1-SPICLK_P-Pad37) -> /MCU/LED_B
- U1 pad 44: unconnected-(U1-MTCK-Pad44) -> /MCU/RAD_BUSY
- U1 pad 45: unconnected-(U1-MTDO-Pad45) -> /MCU/RAD_RF_EN
- U1 pad 47: unconnected-(U1-MTDI-Pad47) -> /MCU/LED_R
- U1 pad 48: unconnected-(U1-MTMS-Pad48) -> /MCU/LED_G
- U1 pad 7: unconnected-(U1-GPIO2-Pad7) -> /MCU/RAD_DIO1
- U9 pad 3: /IO/USB_D+ -> /IO/USB_D-
Routing:
- net +BATT: track 0.00 -> 13.9 mm
- net /IO/CANTX: track 0.00 -> 9.69 mm
- net +3V3: track 0.00 -> 8.29 mm, vias 0 -> 1
- net /IO/CAN_L: track 0.00 -> 7.32 mm
- net /MCU/SPI2_IO3: track 0.00 -> 6.97 mm
- net /MCU/TXD_MCU: track 0.00 -> 6.28 mm
- net /IO/CAN_H: track 0.00 -> 6.15 mm
- net /IO/CANRX: track 0.00 -> 5.72 mm
- net /IO/USB_UNSAFE_D+: track 0.00 -> 5.09 mm
- net /MCU/SPI2_CLK: track 0.00 -> 5.02 mm
- net /MCU/SPI2_IO0: track 0.00 -> 3.58 mm
- net /MCU/RXD_MCU: track 0.00 -> 3.30 mm
- net /IO/BATT_RAW: track 0.00 -> 3.22 mm, vias 0 -> 1
- net Net-(Q1-S): track 0.00 -> 3.02 mm
- net /IO/TXD_MCU: track 0.00 -> 2.98 mm
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- added copper zone on In1.Cu, net +3V3
- added copper zone on In2.Cu, net GND

Commit message: iris inital layout
Parts:
- added D5: BZX584C10, Diode_SMD:D_SOD-523, B.Cu at (108.8, 135.9)
- added R37: 100k, Resistor_SMD:R_0402_1005Metric, B.Cu at (108.8, 137.8)
Connections:
- Q1 pad 3: GND -> Net-(D5-A)

Commit message: for foo & root
Parts:
- added D6: BZX584C10, Diode_SMD:D_SOD-523, B.Cu at (115.2, 132.8)
- added Q11: AO3400A, Package_TO_SOT_SMD:SOT-23, B.Cu at (115.7, 136.0)
- moved R34 8.98 mm to (108.9, 119.5), turned to -90 degrees
- moved R33 7.14 mm to (110.2, 119.5), turned to 90 degrees
- moved C27 1.95 mm to (111.5, 116.7)
- moved C6 1.95 mm to (110.5, 116.7)
- moved R39 1.73 mm to (117.9, 134.2)
- moved R27 1.12 mm to (104.6, 114.9)
- moved R26 1.12 mm to (104.6, 113.9)
- moved C35 0.90 mm to (120.4, 105.6)
- moved U8 0.90 mm to (119.4, 110.5)
- moved R30 0.77 mm to (116.3, 116.4)
- moved R31 0.77 mm to (115.2, 116.4)
- moved C28 0.65 mm to (120.2, 127.5)
- moved J6 0.65 mm to (117.3, 131.8)
- moved U5 0.65 mm to (120.3, 130.4)
- moved C37 0.54 mm to (105.8, 116.8)
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Connections:
- BZ1 pad 1: /MCU/BUZZER -> +3V3
- BZ1 pad 2: GND -> Net-(BZ1--)
Routing:
- net /IO/CANTX: track 9.69 -> 0.00 mm
- net /IO/CAN_L: track 7.32 -> 0.00 mm
- net /MCU/SPI2_IO3: track 6.97 -> 0.00 mm
- net /IO/CAN_H: track 6.15 -> 0.00 mm
- net /IO/CANRX: track 5.72 -> 0.00 mm
- net /IO/USB_UNSAFE_D+: track 5.09 -> 0.00 mm
- net /MCU/SPI2_CLK: track 5.02 -> 0.00 mm
- net /MCU/SPI2_IO0: track 3.58 -> 0.00 mm
- net /IO/USB_UNSAFE_D-: track 2.31 -> 0.00 mm
- net /IO/USB_D-: track 1.97 -> 0.00 mm
- net /IO/USB_D+: track 1.63 -> 0.00 mm
- net +3V3: track 8.29 -> 7.08 mm
- net GND: track 2.86 -> 2.15 mm, vias 2 -> 1

Commit message: routed
Parts:
- added C7: 100n, Capacitor_SMD:C_0402_1005Metric, B.Cu at (104.0, 109.6)
- added R13: 0, Resistor_SMD:R_0603_1608Metric, F.Cu at (117.3, 135.6)
- added R38: 0, Resistor_SMD:R_0402_1005Metric, B.Cu at (117.1, 123.0)
- moved R34 9.34 mm to (115.8, 125.8), turned to 0 degrees
- moved R33 7.57 mm to (115.8, 124.6), turned to 180 degrees
- moved C37 7.35 mm to (104.6, 124.0), turned to 90 degrees
- moved U4 5.17 mm to (106.7, 124.0), turned to 90 degrees
- moved C38 5.13 mm to (103.9, 119.6)
- moved U7 5.13 mm to (106.3, 118.3)
- moved C36 4.93 mm to (105.4, 121.6), turned to 180 degrees
- moved R28 4.11 mm to (114.9, 105.6), turned to 0 degrees
- moved R19 3.95 mm to (114.0, 122.6), turned to -90 degrees
- moved R18 3.07 mm to (113.0, 122.1), turned to -90 degrees
- moved R24 3.00 mm to (104.4, 112.0), turned to 0 degrees
- moved R29 2.69 mm to (114.9, 104.6), turned to 180 degrees
- moved R39 2.62 mm to (120.3, 133.1), turned to 180 degrees
- moved D1 2.38 mm to (112.8, 124.7), turned to 0 degrees
- moved R17 2.10 mm to (112.0, 121.9), turned to -90 degrees
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Connections:
- J3 pad SH: unconnected-(J3-Shield-PadSH)_5 -> Net-(J3-Shield)
- J6 pad 1: /IO/GPIO -> Net-(J6-Pin_1)
- U1 pad 11: /MCU/RAD_RST -> /MCU/RAD_DIO2
- U1 pad 12: /MCU/LSM_INT1 -> /MCU/RAD_DIO1
- U1 pad 13: /MCU/LSM_INT2 -> /MCU/RAD_RST
- U1 pad 38: /MCU/I2C_SDA -> /MCU/LED_R
- U1 pad 39: /MCU/I2C_SCL -> /MCU/LED_G
- U1 pad 43: /IO/GPIO -> unconnected-(U1-GPIO38-Pad43)
- U1 pad 47: /MCU/LED_R -> /MCU/LSM_INT1
- U1 pad 48: /MCU/LED_G -> /MCU/LSM_INT2
- U1 pad 7: /MCU/RAD_DIO1 -> /MCU/RAD_DIO3
- U10 pad 7: unconnected-(U10-DIO2-Pad7) -> /MCU/RAD_DIO2
- U10 pad 8: unconnected-(U10-DIO3-Pad8) -> /MCU/RAD_DIO3
- U4 pad 13: /MCU/I2C_SCL -> /MCU/SPI3_SCLK
- U4 pad 14: /MCU/I2C_SDA -> /MCU/SPI3_COPI
- U4 pad 2: /MCU/SPI3_SCLK -> GND
- U4 pad 3: /MCU/SPI3_COPI -> GND
Routing:
- net GND: track 2.15 -> 52.2 mm, vias 1 -> 33
- net +3V3: track 7.08 -> 53.6 mm, vias 1 -> 21
- net /MCU/RXD_MCU: track 3.30 -> 42.5 mm, vias 0 -> 2
- net /MCU/TXD_MCU: track 6.28 -> 41.2 mm, vias 0 -> 2
- net /MCU/SPI3_CIPO: track 0.00 -> 31.6 mm, vias 0 -> 2
- net /MCU/BUZZER: track 0.00 -> 30.2 mm, vias 0 -> 2
- net /MCU/SPI3_COPI: track 0.00 -> 28.9 mm, vias 0 -> 4
- net /MCU/SPI3_SCLK: track 0.00 -> 28.7 mm, vias 0 -> 2
- net VBUS: track 1.97 -> 28.9 mm, vias 0 -> 3
- net /MCU/VSENSE: track 0.00 -> 24.3 mm, vias 0 -> 2
- net /MCU/MS56_CS: track 0.00 -> 20.2 mm, vias 0 -> 2
- net /MCU/CANTX: track 0.00 -> 17.5 mm
- net /MCU/LSM_INT1: track 0.00 -> 17.0 mm, vias 0 -> 2
- net /MCU/CANRX: track 0.00 -> 16.7 mm
- net /MCU/LSM_CS: track 0.00 -> 16.5 mm, vias 0 -> 4
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- added copper zone on F.Cu, net GND

Commit message: root feedback
Parts:
- added C12: 10u, Capacitor_SMD:C_0805_2012Metric, B.Cu at (112.5, 125.5)
- added R51: 0, Resistor_SMD:R_0402_1005Metric, B.Cu at (117.2, 126.9)
- L5: value L_Small -> 0
- R21: value 1k -> 15k
- R32: value 1k -> 5k
- moved U5 0.10 mm to (120.4, 130.4)
Connections:
- U5 pad 8: unconnected-(U5-STB-Pad8) -> Net-(U5-STB)
Routing:
- net +3V3: track 53.6 -> 60.2 mm, vias 21 -> 23
- net Net-(U5-STB): track 0.00 -> 5.67 mm
- net /MCU/BUZZER: track 30.2 -> 26.1 mm
- net VBUS: track 28.9 -> 33.0 mm
- net /MCU/CANTX: track 17.5 -> 15.6 mm
- net /MCU/SPI3_CIPO: track 31.6 -> 30.3 mm
- net /MCU/GPIO45: track 5.48 -> 6.43 mm
- net /MCU/CANRX: track 16.7 -> 15.9 mm
- net /MCU/RST: track 10.3 -> 11.1 mm, vias 0 -> 1
- net /MCU/RAD_DIO2: track 11.4 -> 10.8 mm
- net Net-(D1-RK): track 1.21 -> 1.86 mm

Commit message: updates from folks
Parts:
- renumbered L5 to Le1
Connections:
- J3 pad 2: /IO/USB_UNSAFE_D- -> /IO/USB_D-
- J3 pad 3: /IO/USB_UNSAFE_D+ -> /IO/USB_D+
- U9 pad 4: /IO/USB_UNSAFE_D- -> /IO/USB_D-
- U9 pad 6: /IO/USB_UNSAFE_D+ -> /IO/USB_D+
Routing:
- net /IO/USB_D+: track 1.69 -> 9.00 mm
- net /IO/USB_UNSAFE_D+: track 5.04 -> 0.00 mm
- net /IO/USB_D-: track 1.78 -> 6.32 mm
- net /IO/USB_UNSAFE_D-: track 2.27 -> 0.00 mm
- net VBUS: track 33.0 -> 31.7 mm, vias 3 -> 4
- net /MCU/SPI3_COPI: track 29.2 -> 30.0 mm

Commit message: witness release
Other:
- board text added: "BATT+"
- board text added: "CAN"
- board text added: "DESIGNED BY: E. SOHN"
- board text added: "NO COMMS?"
- board text added: "NO DATA?"
- board text added: "UART"
- board text added: "WITNESS V1"
- board text added: "made on earth, by humans"
