File: Hardware/witnessv0.2/aperture/aperture.kicad_sch (KiCad schematic)
At the start: 8 parts, among them U1 L80-R, U10 RA-01SH-P

Commit message: aperture ready for order probably
Connections:
- net GPS_RST: no longer A1.9 (IO36/A4)
Other:
- title: (none) -> APERTURE
Changed lines of the file:
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@@
 	(generator_version "10.0")
 	(paper "A4")
+	(title_block
+		(title "APERTURE")
+	)
 	(text "GPS\n"
 		(exclude_from_sim no)
@@
 		)
 		(stroke
-			(width 0)
-			(type default)
-		)
-	)
-	(wire
-		(pts
-			(xy 142.24 132.08) (xy 152.4 132.08)
-		)
-		(stroke
