File: Hardware/witnessv0.2/aperture/aperture.kicad_pcb (KiCad board)
At the start: 2 copper layers, 23 x 51 mm, 8 parts, among them U1 L80-R, U10 RA-01SH-P

Commit message: aperture ready for order probably
Parts:
- moved R2 1.37 mm to (136.8, 72.8), turned to -90 degrees
- moved R1 1.10 mm to (135.1, 72.8)
Routing:
- net /TX_MCU: track 53.2 -> 49.8 mm
- net +3V3: track 62.5 -> 61.2 mm
- net Net-(U1-TXD1): track 3.52 -> 2.42 mm
- net Net-(U1-RXD1): track 3.51 -> 4.33 mm
- net /RX_MCU: track 48.9 -> 48.2 mm
- net GND: vias 62 -> 86
Other:
- board size 23 x 51 mm -> 23.6 x 51 mm
- board text added: "APERTURE GROUND STATION V1"
- board text added: "JLCJLCJLCJLC"

Commit message: aperture release 1
Other:
- board text added: "DESIGNED BY: ELIJAH SOHN IF FOUND CALL 646 618 4415"
- board text added: "no data?"
Changed lines of the file:
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@@
+		)
+	)
+	(gr_text "no data?"
+		(at 129.6 101.9 0)
+		(layer "F.SilkS")
+		(effects
+			(font
+				(size 1 1)
+				(thickness 0.1)
+			)
+			(justify left bottom)
+		)
+	)
+	(gr_text "DESIGNED BY: \nELIJAH SOHN\nIF FOUND CALL\n646 618 4415\n"
+		(at 135.6 101.4 -0)
+		(layer "B.SilkS")
+		(effects
+			(font
+				(size 1 1)
+				(thickness 0.1)
+			)
+			(justify left bottom mirror)
 		)
 	)
 	(gr_text "JLCJLCJLCJLC"
-		(at 139.3 80.5 180)
+		(at 126.4 77.4 180)
 		(layer "B.SilkS")
 		(effects
@@
 				(thickness 0.15)
 			)
-			(justify left bottom)
+			(justify left bottom mirror)
 		)
 	)
